File: ADC_CS5381KKSZ_Board.kicad_sch (KiCad schematic)
At the start: 115 parts, among them IC1 OpAmp_NE5532D, J1 Mode_Selection_Jumpers, J10 JST_XH_2.54_Plug_12V+, J11 JST_XH_2.54_Plug_12V-, J12 I2S_Headers, J13 MCLK_DIV_Jumper, J14 JST_XH_2.54_Plug_5V+, J15 USB_B_Micro, J16 USB_D_Jumper, J17 MCLK_Jumper, J2 JST_XH_2.54_Plug_3V3+, J3 3V3_Power_Selector_Jumper, J4 3V_Selection_Header, J5 I/O_Headers, J6 I2S_OR_LJ_OUT, J7 I2S_OR_LJ_OUT, J8 HP_FILTER_EN, J9 I/O_Headers, Q1 MOSFET_SI2333DDS-T1-BE3, Q2 MOSFET_SI2333DDS-T1-BE3, Q3 MOSFET_SI2343DS-T1-BE3, Q4 MOSFET_SI2343DS-T1-BE3, U1 CS5381

Commit message: Update
Parts:
- J5: footprint Connector_PinHeader_2.54mm:PinHeader_2x05_P2.54mm_Vertical -> Connector_PinHeader_2.54mm:PinHeader_2x05_P2.54mm_Horizontal
Connections:
- net EXT_POWER_12V-_PP renamed EXT_POWER_12V-
Other:
- moved on the sheet: C39, C40, C41, C42, D4, D5
Changed lines of the file:
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@@
 	(wire
 		(pts
-			(xy 410.21 298.45) (xy 410.21 290.83)
+			(xy 410.21 297.18) (xy 410.21 290.83)
 		)
 		(stroke
@@
 	(wire
 		(pts
-			(xy 387.35 287.02) (xy 387.35 290.83)
+			(xy 387.35 285.75) (xy 387.35 290.83)
 		)
 		(stroke
@@
 	(wire
 		(pts
-			(xy 420.37 290.83) (xy 420.37 298.45)
+			(xy 420.37 290.83) (xy 420.37 297.18)
 		)
 		(stroke
@@
 	(wire
 		(pts
-			(xy 387.35 290.83) (xy 387.35 297.18)
+			(xy 387.35 290.83) (xy 387.35 295.91)
 		)
 		(stroke
@@
 	(wire
 		(pts
-			(xy 420.37 306.07) (xy 420.37 308.61)
+			(xy 420.37 304.8) (xy 420.37 308.61)
 		)
 		(stroke
@@
 	(wire
 		(pts
-			(xy 387.35 304.8) (xy 387.35 308.61)
+			(xy 387.35 303.53) (xy 387.35 308.61)
 		)
 		(stroke
@@
 	(wire
 		(pts
-			(xy 420.37 287.02) (xy 420.37 290.83)
+			(xy 420.37 285.75) (xy 420.37 290.83)
 		)
 		(stroke
@@
 	(wire
 		(pts
-			(xy 387.35 273.05) (xy 387.35 279.4)
+			(xy 387.35 273.05) (xy 387.35 278.13)
 		)
 		(stroke
@@
 	(wire
 		(pts
-			(xy 420.37 273.05) (xy 420.37 279.4)
+			(xy 420.37 273.05) (xy 420.37 278.13)
 		)
 		(stroke
@@
 	(wire
 		(pts
-			(xy 410.21 306.07) (xy 410.21 308.61)
+			(xy 410.21 304.8) (xy 410.21 308.61)
 		)
 		(stroke
@@
 	(wire
 		(pts
-			(xy 410.21 287.02) (xy 410.21 290.83)
+			(xy 410.21 285.75) (xy 410.21 290.83)
 		)
 		(stroke
@@
 	(wire
 		(pts
-			(xy 410.21 279.4) (xy 410.21 273.05)
+			(xy 410.21 278.13) (xy 410.21 273.05)
 		)
 		(stroke
@@
 	(label "MIC_L_OUTPUT-"
 		(at 83.82 101.6 270)
+		(fields_autoplaced yes)
 		(effects
 			(font
@@
 	(label "IN-"
 		(at 133.35 60.96 180)
+		(fields_autoplaced yes)
 		(effects
 			(font
@@
 	(label "LT1128CS8_L1_IN+"
 		(at 130.81 71.12 180)
+		(fields_autoplaced yes)
 		(effects
 			(font
@@
 	(label "IN-"
 		(at 134.62 125.73 180)
+		(fields_autoplaced yes)
 		(effects
 			(font
@@
 	(label "IN-"
 		(at 316.23 59.69 180)
+		(fields_autoplaced yes)
 		(effects
 			(font
@@
 	(label "MIC_L_OUTPUT+"
 		(at 83.82 99.06 90)
+		(fields_autoplaced yes)
 		(effects
 			(font
@@
 	(label "LT1128CS8_R2_IN+"
 		(at 309.88 134.62 180)
+		(fields_autoplaced yes)
 		(effects
 			(font
@@
 	(label "LT1128CS8_L2_IN+"
 		(at 130.81 135.89 180)
+		(fields_autoplaced yes)
 		(effects
 			(font
@@
 	(label "IN-"
 		(at 317.5 124.46 180)
+		(fields_autoplaced yes)
 		(effects
 			(font
@@
 	(label "LT1128CS8_R1_IN+"
 		(at 311.15 69.85 180)
+		(fields_autoplaced yes)
 		(effects
 			(font
@@
 		)
 	)
-	(label "EXT_POWER_12V-_PP"
+	(label "EXT_POWER_12V-"
 		(at 312.42 303.53 0)
 		(fields_autoplaced yes)
@@
 	(symbol
 		(lib_id "Device:C_Polarized")
-		(at 410.21 283.21 0)
+		(at 410.21 281.94 0)
 		(unit 1)
 		(exclude_from_sim no)
@@
 		(dnp no)
 		(property "Reference" "C39"
-			(at 408.178 286.512 90)
+			(at 408.178 285.242 90)
 			(effects
 				(font
@@
 		)
 		(property "Value" "47u"
-			(at 408.432 278.13 90)
+			(at 408.432 276.86 90)
 			(effects
 				(font
@@
 		)
 		(property "Footprint" "Capacitor_SMD:C_0805_2012Metric"
-			(at 411.1752 287.02 0)
+			(at 411.1752 285.75 0)
 			(effects
 				(font
@@
 		)
 		(property "Datasheet" "~"
-			(at 410.21 283.21 0)
+			(at 410.21 281.94 0)
 			(effects
 				(font
@@
 		)
 		(property "Description" "Polarized capacitor"
-			(at 410.21 283.21 0)
+			(at 410.21 281.94 0)
 			(effects
 				(font
@@
 	(symbol
 		(lib_id "Device:C")
-		(at 420.37 283.21 0)
+		(at 420.37 281.94 0)
 		(unit 1)
 		(exclude_from_sim no)
@@
 		(dnp no)
 		(property "Reference" "C40"
-			(at 421.386 280.924 0)
+			(at 421.386 279.654 0)
 			(effects
 				(font
@@
 		)
 		(property "Value" "10n_X7R"
-			(at 421.64 285.496 0)
+			(at 421.64 284.226 0)
 			(effects
 				(font
@@
 		)
 		(property "Footprint" "Capacitor_SMD:C_0805_2012Metric"
-			(at 421.3352 287.02 0)
+			(at 421.3352 285.75 0)
 			(effects
 				(font
@@
 		)
 		(property "Datasheet" "~"
-			(at 420.37 283.21 0)
+			(at 420.37 281.94 0)
 			(effects
 				(font
@@
 		)
 		(property "Description" "Unpolarized capacitor"
-			(at 420.37 283.21 0)
+			(at 420.37 281.94 0)
 			(effects
 				(font
@@
 			)
 		)
-		(property "Footprint" "Connector_PinHeader_2.54mm:PinHeader_2x05_P2.54mm_Vertical"
+		(property "Footprint" "Connector_PinHeader_2.54mm:PinHeader_2x05_P2.54mm_Horizontal"
 			(at 388.62 190.5 0)
 			(effects
@@
 	(symbol
 		(lib_id "Diode:BZX84Cxx")
-		(at 387.35 283.21 270)
+		(at 387.35 281.94 270)
 		(unit 1)
 		(exclude_from_sim no)
@@
 		(fields_autoplaced yes)
 		(property "Reference" "D4"
-			(at 389.89 281.9399 90)
+			(at 389.89 280.6699 90)
 			(effects
 				(font
@@
 		)
 		(property "Value" "BZX84C13LT1G"
-			(at 389.89 284.4799 90)
+			(at 389.89 283.2099 90)
 			(effects
 				(font
@@
 		)
 		(property "Footprint" "Package_TO_SOT_SMD:SOT-23"
-			(at 387.35 283.21 0)
+			(at 387.35 281.94 0)
 			(effects
 				(font
@@
 		)
 		(property "Datasheet" "https://diotec.com/tl_files/diotec/files/pdf/datasheets/bzx84c2v4.pdf"
-			(at 387.35 283.21 0)
+			(at 387.35 281.94 0)
 			(effects
 				(font
@@
 		)
 		(property "Description" "300mW Zener Diode, SOT-23"
-			(at 387.35 283.21 0)
+			(at 387.35 281.94 0)
 			(effects
 				(font
@@
 	(symbol
 		(lib_id "Device:C_Polarized")
-		(at 410.21 302.26 0)
+		(at 410.21 300.99 0)
 		(unit 1)
 		(exclude_from_sim no)
@@
 		(dnp no)
 		(property "Reference" "C41"
-			(at 408.178 305.562 90)
+			(at 408.178 304.292 90)
 			(effects
 				(font
@@
 		)
 		(property "Value" "47u"
-			(at 408.432 297.18 90)
+			(at 408.432 295.91 90)
 			(effects
 				(font
@@
 		)
 		(property "Footprint" "Capacitor_SMD:C_0805_2012Metric"
-			(at 411.1752 306.07 0)
+			(at 411.1752 304.8 0)
 			(effects
 				(font
@@
 		)
 		(property "Datasheet" "~"
-			(at 410.21 302.26 0)
+			(at 410.21 300.99 0)
 			(effects
 				(font
@@
 		)
 		(property "Description" "Polarized capacitor"
-			(at 410.21 302.26 0)
+			(at 410.21 300.99 0)
 			(effects
 				(font
@@
 	(symbol
 		(lib_id "Diode:BZX84Cxx")
-		(at 387.35 300.99 270)
+		(at 387.35 299.72 270)
 		(unit 1)
 		(exclude_from_sim no)
@@
 		(fields_autoplaced yes)
 		(property "Reference" "D5"
-			(at 389.89 299.7199 90)
+			(at 389.89 298.4499 90)
 			(effects
 				(font
@@
 		)
 		(property "Value" "BZX84C13LT1G"
-			(at 389.89 302.2599 90)
+			(at 389.89 300.9899 90)
 			(effects
 				(font
@@
 		)
 		(property "Footprint" "Package_TO_SOT_SMD:SOT-23"
-			(at 387.35 300.99 0)
+			(at 387.35 299.72 0)
 			(effects
 				(font
@@
 		)
 		(property "Datasheet" "https://diotec.com/tl_files/diotec/files/pdf/datasheets/bzx84c2v4.pdf"
-			(at 387.35 300.99 0)
+			(at 387.35 299.72 0)
 			(effects
 				(font
@@
 		)
 		(property "Description" "300mW Zener Diode, SOT-23"
-			(at 387.35 300.99 0)
+			(at 387.35 299.72 0)
 			(effects
 				(font
@@
 	(symbol
 		(lib_id "Device:C")
-		(at 420.37 302.26 0)
+		(at 420.37 300.99 0)
 		(unit 1)
 		(exclude_from_sim no)
@@
 		(dnp no)
 		(property "Reference" "C42"
-			(at 421.386 299.974 0)
+			(at 421.386 298.704 0)
 			(effects
 				(font
@@
 		)
 		(property "Value" "10n_X7R"
-			(at 421.64 304.546 0)
+			(at 421.64 303.276 0)
 			(effects
 				(font
@@
 		)
 		(property "Footprint" "Capacitor_SMD:C_0805_2012Metric"
-			(at 421.3352 306.07 0)
+			(at 421.3352 304.8 0)
 			(effects
 				(font
@@
 		)
 		(property "Datasheet" "~"
-			(at 420.37 302.26 0)
+			(at 420.37 300.99 0)
 			(effects
 				(font
@@
 		)
 		(property "Description" "Unpolarized capacitor"
-			(at 420.37 302.26 0)
+			(at 420.37 300.99 0)
 			(effects
 				(font

Commit message: Update
Connections:
- removed net IN-: C10.1, C16.1, C19.1, C9.1, OA1.2 (IN-), OA2.2 (IN-), OA3.2 (IN-), OA4.2 (IN-), R13.1, R14.1, R6.1, R7.1
- new net L1_IN-: C9.1, OA1.2 (IN-), R6.1
- new net L2_IN-: C10.1, OA2.2 (IN-), R7.1
- new net R1_IN-: C16.1, OA3.2 (IN-), R13.1
- new net R2_IN-: C19.1, OA4.2 (IN-), R14.1
Changed lines of the file:
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@@
 	)
 	(junction
+		(at 308.61 34.29)
+		(diameter 0)
+		(color 0 0 0 0)
+	)
+	(junction
 		(at 182.88 130.81)
 		(diameter 0)
@@
 	)
 	(junction
-		(at 311.15 34.29)
-		(diameter 0)
-		(color 0 0 0 0)
-	)
-	(junction
 		(at 271.78 69.85)
 		(diameter 0)
@@
 	)
 	(junction
-		(at 128.27 35.56)
-		(diameter 0)
-		(color 0 0 0 0)
-	)
-	(junction
 		(at 398.78 187.96)
 		(diameter 0)
@@
 	)
 	(junction
-		(at 312.42 99.06)
-		(diameter 0)
-		(color 0 0 0 0)
-	)
-	(junction
 		(at 353.06 129.54)
 		(diameter 0)
@@
 	)
 	(junction
+		(at 125.73 100.33)
+		(diameter 0)
+		(color 0 0 0 0)
+	)
+	(junction
 		(at 375.92 273.05)
 		(diameter 0)
@@
 	)
 	(junction
-		(at 129.54 100.33)
-		(diameter 0)
-		(color 0 0 0 0)
-	)
-	(junction
 		(at 410.21 308.61)
 		(diameter 0)
@@
 	)
 	(junction
+		(at 125.73 35.56)
+		(diameter 0)
+		(color 0 0 0 0)
+	)
+	(junction
 		(at 351.79 64.77)
 		(diameter 0)
@@
 	)
 	(junction
+		(at 309.88 99.06)
+		(diameter 0)
+		(color 0 0 0 0)
+	)
+	(junction
 		(at 463.55 119.38)
 		(diameter 0)
@@
 	(wire
 		(pts
-			(xy 326.39 34.29) (xy 311.15 34.29)
-		)
-		(stroke
-			(width 0)
-			(type default)
-		)
-	)
-	(wire
-		(pts
 			(xy 99.06 255.27) (xy 101.6 255.27)
 		)
@@
 	(wire
 		(pts
-			(xy 311.15 27.94) (xy 311.15 34.29)
+			(xy 308.61 27.94) (xy 308.61 34.29)
 		)
 		(stroke
@@
 	(wire
 		(pts
-			(xy 312.42 99.06) (xy 312.42 124.46)
+			(xy 309.88 99.06) (xy 309.88 124.46)
 		)
 		(stroke
@@
 	(wire
 		(pts
-			(xy 326.39 27.94) (xy 311.15 27.94)
+			(xy 326.39 27.94) (xy 308.61 27.94)
 		)
 		(stroke
@@
 	(wire
 		(pts
-			(xy 311.15 34.29) (xy 311.15 59.69)
+			(xy 308.61 34.29) (xy 308.61 59.69)
 		)
 		(stroke
@@
 	(wire
 		(pts
-			(xy 128.27 29.21) (xy 128.27 35.56)
+			(xy 125.73 29.21) (xy 125.73 35.56)
 		)
 		(stroke
@@
 	(wire
 		(pts
-			(xy 128.27 35.56) (xy 128.27 60.96)
+			(xy 125.73 35.56) (xy 125.73 60.96)
 		)
 		(stroke
@@
 	(wire
 		(pts
-			(xy 105.41 104.14) (xy 124.46 104.14)
+			(xy 105.41 104.14) (xy 120.65 104.14)
 		)
 		(stroke
@@
 	(wire
 		(pts
-			(xy 144.78 100.33) (xy 129.54 100.33)
+			(xy 125.73 100.33) (xy 144.78 100.33)
 		)
 		(stroke
@@
 	(wire
 		(pts
-			(xy 119.38 214.63) (xy 119.38 219.71)
+			(xy 125.73 35.56) (xy 143.51 35.56)
 		)
 		(stroke
@@
 	(wire
 		(pts
-			(xy 340.36 186.69) (xy 342.9 186.69)
+			(xy 119.38 214.63) (xy 119.38 219.71)
 		)
 		(stroke
@@
 	(wire
 		(pts
-			(xy 454.66 44.45) (xy 454.66 49.53)
+			(xy 340.36 186.69) (xy 342.9 186.69)
 		)
 		(stroke
@@
 	(wire
 		(pts
-			(xy 387.35 290.83) (xy 387.35 295.91)
+			(xy 454.66 44.45) (xy 454.66 49.53)
 		)
 		(stroke
@@
 	(wire
 		(pts
-			(xy 396.24 195.58) (xy 398.78 195.58)
+			(xy 387.35 290.83) (xy 387.35 295.91)
 		)
 		(stroke
@@
 	(wire
 		(pts
-			(xy 344.17 278.13) (xy 354.33 278.13)
+			(xy 396.24 195.58) (xy 398.78 195.58)
 		)
 		(stroke
@@
 	(wire
 		(pts
-			(xy 490.22 234.95) (xy 513.08 234.95)
+			(xy 344.17 278.13) (xy 354.33 278.13)
 		)
 		(stroke
@@
 	(wire
 		(pts
-			(xy 327.66 99.06) (xy 312.42 99.06)
+			(xy 490.22 234.95) (xy 513.08 234.95)
 		)
 		(stroke
@@
 	(wire
 		(pts
-			(xy 129.54 100.33) (xy 129.54 125.73)
+			(xy 125.73 100.33) (xy 125.73 125.73)
 		)
 		(stroke
@@
 	(wire
 		(pts
-			(xy 143.51 29.21) (xy 128.27 29.21)
+			(xy 143.51 29.21) (xy 125.73 29.21)
 		)
 		(stroke
@@
 	(wire
 		(pts
-			(xy 327.66 92.71) (xy 312.42 92.71)
+			(xy 327.66 92.71) (xy 309.88 92.71)
 		)
 		(stroke
@@
 	(wire
 		(pts
+			(xy 308.61 34.29) (xy 326.39 34.29)
+		)
+		(stroke
+			(width 0)
+			(type default)
+		)
+	)
+	(wire
+		(pts
 			(xy 198.12 370.84) (xy 198.12 373.38)
 		)
@@
 	(wire
 		(pts
-			(xy 129.54 125.73) (xy 134.62 125.73)
+			(xy 125.73 125.73) (xy 134.62 125.73)
 		)
 		(stroke
@@
 	(wire
 		(pts
-			(xy 312.42 92.71) (xy 312.42 99.06)
+			(xy 309.88 92.71) (xy 309.88 99.06)
 		)
 		(stroke
@@
 	(wire
 		(pts
-			(xy 128.27 60.96) (xy 133.35 60.96)
+			(xy 125.73 60.96) (xy 133.35 60.96)
 		)
 		(stroke
@@
 	(wire
 		(pts
-			(xy 129.54 93.98) (xy 129.54 100.33)
+			(xy 125.73 93.98) (xy 125.73 100.33)
 		)
 		(stroke
@@
 	(wire
 		(pts
-			(xy 144.78 93.98) (xy 129.54 93.98)
+			(xy 144.78 93.98) (xy 125.73 93.98)
 		)
 		(stroke
@@
 	(wire
 		(pts
-			(xy 143.51 35.56) (xy 128.27 35.56)
-		)
-		(stroke
-			(width 0)
-			(type default)
-		)
-	)
-	(wire
-		(pts
 			(xy 113.03 219.71) (xy 113.03 236.22)
 		)
@@
 	(wire
 		(pts
-			(xy 311.15 59.69) (xy 316.23 59.69)
+			(xy 308.61 59.69) (xy 316.23 59.69)
 		)
 		(stroke
@@
 	(wire
 		(pts
+			(xy 309.88 99.06) (xy 327.66 99.06)
+		)
+		(stroke
+			(width 0)
+			(type default)
+		)
+	)
+	(wire
+		(pts
 			(xy 129.54 177.8) (xy 129.54 180.34)
 		)
@@
 	(wire
 		(pts
-			(xy 312.42 124.46) (xy 317.5 124.46)
+			(xy 309.88 124.46) (xy 317.5 124.46)
 		)
 		(stroke
@@
 		)
 	)
-	(label "IN-"
+	(label "L1_IN-"
 		(at 133.35 60.96 180)
 		(fields_autoplaced yes)
@@
 		)
 	)
-	(label "IN-"
+	(label "L2_IN-"
 		(at 134.62 125.73 180)
 		(fields_autoplaced yes)
@@
 		)
 	)
-	(label "IN-"
+	(label "R1_IN-"
 		(at 316.23 59.69 180)
 		(fields_autoplaced yes)
@@
 		)
 	)
-	(label "IN-"
+	(label "R2_IN-"
 		(at 317.5 124.46 180)
 		(fields_autoplaced yes)
@@
 	)
 	(label "VCOM_B_LEFT"
-		(at 124.46 104.14 180)
+		(at 120.65 104.14 180)
 		(fields_autoplaced yes)
 		(effects

Commit message: Update
Other:
- note added: "STM32MP157FAD1 TFBGA257 Pitch 0.5 2x STM32WB55CGU6 2x STM32WB5MMGH6TR STM32MP135DAF7 TFBGA320 Pitch 0.5 STM32H7S7L8H6H TFBGA 225 0.8 mm pitch STSPIN958TR STM32H7S3I8T6 LSM6DSV16XTR ISM330BXTR STM32WL55CCU6 STM32WL55JCI6 2x STM32MP157DAA1 2x LFBGA448 Pitch: 0.8 mm AGVLB.25B.07.0060A Connector: I-PEX MHF® I (U.FL Compatible) GW.52.A153 2.4/5.8/7.1GHZ Hinged RP-SMA (M) Connector TI.96.A113 900-940MH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"
Changed lines of the file:
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@@
+		)
+	)
+	(text "STM32MP157FAD1 TFBGA257 Pitch 0.5 2x\nSTM32WB55CGU6 2x\nSTM32WB5MMGH6TR\nSTM32MP135DAF7 TFBGA320 Pitch 0.5\nSTM32H7S7L8H6H TFBGA 225 0.8 mm pitch\n\nSTSPIN958TR\nSTM32H7S3I8T6\nLSM6DSV16XTR\nISM330BXTR\nSTM32WL55CCU6\nSTM32WL55JCI6 2x\n\nSTM32MP157DAA1 2x LFBGA448 Pitch: 0.8 mm\n\nAGVLB.25B.07.0060A Connector: I-PEX MHF® I (U.FL Compatible)\nGW.52.A153 2.4/5.8/7.1GHZ Hinged RP-SMA (M) Connector\nTI.96.A113 900-940MHZ Connector: SMA(M)\n\nCS5381K-KSZ IC 120DB 192KHZ MULTI-BIT ADC 2x\n\nR9A07G044L28GBG#BC0 2x 551-LFBGA (21x21) pitch 0.8mm\n\nNXP FS32V234CTN2VUB 1x\nNXP MIMXRT1172DVMAA 2x 289-pin MAPBGA, 14 x 14 mm, 0.8 mm pitch"
+		(exclude_from_sim no)
+		(at -53.848 32.004 0)
+		(effects
+			(font
+				(size 1 1)
+			)
+			(justify left)
 		)
 	)

Commit message: Update
Parts:
- removed J12: I2S_Headers, Connector_PinHeader_2.54mm:PinHeader_2x04_P2.54mm_Horizontal, symbol Connector_Generic:Conn_02x04_Odd_Even
- added J12: I2S_Headers, Connector_PinHeader_2.54mm:PinHeader_2x03_P2.54mm_Horizontal, symbol Connector_Generic:Conn_02x03_Odd_Even
Connections:
- net GND: now also J12.2 (Pin_2), J12.3 (Pin_3), J12.6 (Pin_6)
- net LRCK: now also J12.5 (Pin_5)
- net SCLK: now also J12.4 (Pin_4)
- net SDOUT: now also J12.1 (Pin_1)

Commit message: Update
Other:
- note removed: "STM32MP157FAD1 TFBGA257 Pitch 0.5 2x STM32WB55CGU6 2x STM32WB5MMGH6TR STM32MP135DAF7 TFBGA320 Pitch 0.5 STM32H7S7L8H6H TFBGA 225 0.8 mm pitch STSPIN958TR STM32H7S3I8T6 LSM6DSV16XTR ISM330BXTR STM32WL55CCU6 STM32WL55JCI6 2x STM32MP157DAA1 2x LFBGA448 Pitch: 0.8 mm AGVLB.25B.07.0060A Connector: I-PEX MHF® I (U.FL Compatible) GW.52.A153 2.4/5.8/7.1GHZ Hinged RP-SMA (M) Connector TI.96.A113 900-940MH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"
- company: (none) -> Peter Hancak
- title: (none) -> ADC CS5381 Board
Changed lines of the file:
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@@
 	(generator_version "8.0")
 	(paper "A2")
+	(title_block
+		(title "ADC CS5381 Board")
+		(date "2025-07-29")
+		(rev "A")
+		(company "Peter Hancak")
+	)
 	(junction
 		(at 190.5 201.93)
@@
 		)
 	)
-	(text "STM32MP157FAD1 TFBGA257 Pitch 0.5 2x\nSTM32WB55CGU6 2x\nSTM32WB5MMGH6TR\nSTM32MP135DAF7 TFBGA320 Pitch 0.5\nSTM32H7S7L8H6H TFBGA 225 0.8 mm pitch\n\nSTSPIN958TR\nSTM32H7S3I8T6\nLSM6DSV16XTR\nISM330BXTR\nSTM32WL55CCU6\nSTM32WL55JCI6 2x\n\nSTM32MP157DAA1 2x LFBGA448 Pitch: 0.8 mm\n\nAGVLB.25B.07.0060A Connector: I-PEX MHF® I (U.FL Compatible)\nGW.52.A153 2.4/5.8/7.1GHZ Hinged RP-SMA (M) Connector\nTI.96.A113 900-940MHZ Connector: SMA(M)\n\nCS5381K-KSZ IC 120DB 192KHZ MULTI-BIT ADC 2x\n\nR9A07G044L28GBG#BC0 2x 551-LFBGA (21x21) pitch 0.8mm\n\nNXP FS32V234CTN2VUB 1x\nNXP MIMXRT1172DVMAA 2x 289-pin MAPBGA, 14 x 14 mm, 0.8 mm pitch"
-		(exclude_from_sim no)
-		(at -53.848 32.004 0)
-		(effects
-			(font
-				(size 1 1)
-			)
-			(justify left)
-		)
-	)
