File: ADC_CS5381KKSZ_Board.kicad_sch (KiCad schematic)
At the start: 3 parts

Commit message: Update
Changed lines of the file:
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@@
 	(wire
 		(pts
-			(xy 93.98 130.81) (xy 90.17 130.81)
+			(xy 93.98 130.175) (xy 89.535 130.175)
 		)
 		(stroke
@@
 	(wire
 		(pts
-			(xy 96.52 128.27) (xy 90.17 128.27)
-		)
-		(stroke
-			(width 0)
-			(type default)
-		)
-	)
-	(wire
-		(pts
-			(xy 93.98 87.63) (xy 93.98 130.81)
+			(xy 96.52 127.635) (xy 89.535 127.635)
+		)
+		(stroke
+			(width 0)
+			(type default)
+		)
+	)
+	(wire
+		(pts
+			(xy 93.98 87.63) (xy 93.98 130.175)
 		)
 		(stroke
@@
 	(wire
 		(pts
-			(xy 99.06 85.09) (xy 99.06 133.35)
+			(xy 99.06 85.09) (xy 99.06 132.715)
 		)
 		(stroke
@@
 	(wire
 		(pts
-			(xy 96.52 85.09) (xy 96.52 128.27)
-		)
-		(stroke
-			(width 0)
-			(type default)
-		)
-	)
-	(wire
-		(pts
-			(xy 99.06 133.35) (xy 90.17 133.35)
+			(xy 96.52 85.09) (xy 96.52 127.635)
+		)
+		(stroke
+			(width 0)
+			(type default)
+		)
+	)
+	(wire
+		(pts
+			(xy 99.06 132.715) (xy 89.535 132.715)
 		)
 		(stroke
@@
 	)
 	(sheet
-		(at 50.165 123.825)
+		(at 49.53 123.19)
 		(size 40.005 40.64)
 		(fields_autoplaced yes)
@@
 		)
 		(property "Sheetname" "Power_Management"
-			(at 50.165 123.1134 0)
+			(at 49.53 122.4784 0)
 			(effects
 				(font
@@
 		)
 		(property "Sheetfile" "Power_Management.kicad_sch"
-			(at 50.165 165.0496 0)
+			(at 49.53 164.4146 0)
 			(effects
 				(font
@@
 		)
 		(pin "VCOM_B_LEFT" bidirectional
-			(at 90.17 128.27 0)
+			(at 89.535 127.635 0)
 			(effects
 				(font
@@
 		)
 		(pin "VQ_NE5532D" bidirectional
-			(at 90.17 133.35 0)
+			(at 89.535 132.715 0)
 			(effects
 				(font
@@
 		)
 		(pin "VCOM_B_RIGHT" bidirectional
-			(at 90.17 130.81 0)
-			(effects
-				(font
+			(at 89.535 130.175 0)
+			(effects
+				(font

Commit message: Update
Other:
- sheet Interfaces ports: added *RST; removed ~{DISABLE1}_ADA4940, ~{DISABLE2}_ADA4940, ~{RST}_CS5381
- sheet Power_Management ports: added *RST; removed none

Commit message: Update
Connections:
- no-connect marks 0 -> 1
Other:
- sheet Interfaces ports: added I2S1_CK, I2S1_MCK, I2S1_SDI/O, I2S1_WS; removed LRCK, SCLK, SDOUT

Commit message: Update
Parts:
- removed C29: 1uF, Capacitor_SMD:C_0805_2012Metric, symbol Device:C
- removed R22: 5k1, Resistor_SMD:R_0805_2012Metric, symbol Device:R
- removed U2: ~, Personal_Project:Button_KMR231GLFS, symbol Personal_Projects:Button_KMR231GLFS
Other:
- note removed: "RST - Enters low power modde when LOW"

Commit message: Update
Other:
- sheet ADC_CS5381K-KSZ ports: added I2S_LRCK, I2S_SCLK, I2S_SDOUT; removed LRCK, SCLK, SDOUT
Changed lines of the file:
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@@
 		)
 		(fill
-			(color 0 255 255 1.0000)
+			(color 0 132 132 1.0000)
 		)
 		(property "Sheetname" "Interfaces"
@@
 		)
 		(fill
-			(color 0 255 255 1.0000)
+			(color 0 132 132 1.0000)
 		)
 		(property "Sheetname" "ADC_CS5381K-KSZ"
@@
 			)
 		)
-		(pin "SDOUT" bidirectional
-			(at 166.37 54.61 0)
-			(effects
-				(font
-					(size 1.27 1.27)
-				)
-				(justify right)
-			)
-		)
 		(pin "AINR+" bidirectional
 			(at 115.57 54.61 180)
@@
 			)
 		)
-		(pin "SCLK" bidirectional
-			(at 166.37 57.15 0)
-			(effects
-				(font
-					(size 1.27 1.27)
-				)
-				(justify right)
-			)
-		)
-		(pin "LRCK" bidirectional
-			(at 166.37 59.69 0)
-			(effects
-				(font
-					(size 1.27 1.27)
-				)
-				(justify right)
-			)
-		)
 		(pin "M{slash}~{S}" bidirectional
 			(at 166.37 82.55 0)
@@
 			(effects
 				(font
+					(size 1.27 1.27)
+				)
+				(justify right)
+			)
+		)
+		(pin "I2S_SDOUT" bidirectional
+			(at 166.37 54.61 0)
+			(effects
+				(font
+					(size 1.27 1.27)
+				)
+				(justify right)
+			)
+		)
+		(pin "I2S_SCLK" bidirectional
+			(at 166.37 57.15 0)
+			(effects
+				(font
+					(size 1.27 1.27)
+				)
+				(justify right)
+			)
+		)
+		(pin "I2S_LRCK" bidirectional
+			(at 166.37 59.69 0)
+			(effects
+				(font

Commit message: Update
Other:
- sheet ADC_CS5381K-KSZ ports: added none; removed I2S/~{LJ}, MDIV, M/~{S}
- sheet Interfaces ports: added none; removed I2S/~{LJ}, MDIV, M/~{S}
Changed lines of the file:
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@@
-	(wire
-		(pts
-			(xy 166.37 85.09) (xy 194.31 85.09)
-		)
-		(stroke
-			(width 0)
-			(type default)
-		)
-	)
 	(wire
 		(pts
@@
 	(wire
 		(pts
-			(xy 166.37 82.55) (xy 194.31 82.55)
-		)
-		(stroke
-			(width 0)
-			(type default)
-		)
-	)
-	(wire
-		(pts
 			(xy 96.52 129.54) (xy 91.44 129.54)
 		)
@@
 		(pts
 			(xy 90.17 76.2) (xy 101.6 76.2)
-		)
-		(stroke
-			(width 0)
-			(type default)
-		)
-	)
-	(wire
-		(pts
-			(xy 166.37 80.01) (xy 194.31 80.01)
 		)
 		(stroke
@@
 			)
 		)
-		(pin "MDIV" bidirectional
-			(at 194.31 85.09 180)
-			(effects
-				(font
-					(size 1.27 1.27)
-				)
-				(justify left)
-			)
-		)
 		(pin "M1" bidirectional
 			(at 194.31 74.93 180)
@@
 		(pin "~{OVFL}" bidirectional
 			(at 194.31 69.85 180)
-			(effects
-				(font
-					(size 1.27 1.27)
-				)
-				(justify left)
-			)
-		)
-		(pin "I2S{slash}~{LJ}" bidirectional
-			(at 194.31 80.01 180)
-			(effects
-				(font
-					(size 1.27 1.27)
-				)
-				(justify left)
-			)
-		)
-		(pin "M{slash}~{S}" bidirectional
-			(at 194.31 82.55 180)
 			(effects
 				(font
@@
 			)
 		)
-		(pin "MDIV" bidirectional
-			(at 166.37 85.09 0)
-			(effects
-				(font
-					(size 1.27 1.27)
-				)
-				(justify right)
-			)
-		)
 		(pin "VQ_NE5532D" bidirectional
 			(at 115.57 85.09 180)
@@
 			(effects
 				(font
-					(size 1.27 1.27)
-				)
-				(justify right)
-			)
-		)
-		(pin "M{slash}~{S}" bidirectional
-			(at 166.37 82.55 0)
-			(effects
-				(font
-					(size 1.27 1.27)
-				)
-				(justify right)
-			)
-		)
-		(pin "I2S{slash}~{LJ}" bidirectional
-			(at 166.37 80.01 0)
-			(effects
-				(font

Commit message: Update
Other:
- added sheet Notes (Notes.kicad_sch)
- sheet ADC_Driver_ADA4940-2ACPZ-R7 ports: added DP1_HVC/A0, DP1_SCL, DP1_SDA, DP2_HVC/A0, DP2_SCL, DP2_SDA; removed none
- sheet Interfaces ports: added DP1_HVC/A0, DP2_HVC/A0, I2C_SCL_HDR, I2C_SDA_HDR; removed none
- note removed: "Fullscale Input Level = (Ain+)-(Ain-) = 5.64 Vpp Ain+ is between 3.91 and 1.09 V (Each leg swinging 2.82V) Ain- is between 3.91 and 1.09 V Both oscillate around 2.5V (Common mode level) The DC bias (Common mode level) is sett using VQ or VCOM (one pin) VQ or VCOM nominal voltage is 2.5V Filt+ Nominal Voltage 5V (Positive voltage reference output)"
