File: ADC_CS5381KKSZ_Board.kicad_pcb (KiCad board)
At the start: 4 copper layers, 115 parts, among them IC1 OpAmp_NE5532D, J1 Mode_Selection_Jumpers, J10 JST_XH_2.54_Plug_12V+, J11 JST_XH_2.54_Plug_12V-, J12 I2S_Headers, J13 MCLK_DIV_Jumper, J14 JST_XH_2.54_Plug_5V+, J15 USB_B_Micro, J16 USB_D_Jumper, J17 MCLK_Jumper, J2 JST_XH_2.54_Plug_3V3+, J3 3V3_Power_Selector_Jumper, J4 3V_Selection_Header, J5 I/O_Headers, J6 I2S_OR_LJ_OUT, J7 I2S_OR_LJ_OUT, J8 HP_FILTER_EN, J9 I/O_Headers, Q1 MOSFET_SI2333DDS-T1-BE3, Q2 MOSFET_SI2333DDS-T1-BE3, Q3 MOSFET_SI2343DS-T1-BE3, Q4 MOSFET_SI2343DS-T1-BE3, U1 CS5381

Commit message: Update
Parts:
- J5: footprint Connector_PinHeader_2.54mm:PinHeader_2x05_P2.54mm_Vertical -> Connector_PinHeader_2.54mm:PinHeader_2x05_P2.54mm_Horizontal
- moved D1 159.1 mm to (101.9, 28.6)
- moved D3 159.1 mm to (101.9, 33.2)
- moved D4 159.1 mm to (101.9, 37.8)
- moved D5 159.1 mm to (101.9, 42.4)
- moved D6 159.1 mm to (101.9, 47.0)
- moved Q3 159.1 mm to (100.0, 63.0)
- moved H3 159.0 mm to (74.0, 96.0)
- moved Q1 158.7 mm to (91.0, 63.0)
- moved Q4 157.0 mm to (107.0, 64.0)
- moved H1 152.1 mm to (74.0, 54.0)
- moved J4 147.9 mm to (83.0, 62.9)
- moved J10 140.1 mm to (97.7, 59.3)
- moved J11 140.1 mm to (107.0, 59.3)
- moved J14 140.1 mm to (116.2, 59.3)
- moved J2 140.1 mm to (88.5, 59.3)
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Connections:
- net Net-(MK1-OUTPUT+) renamed /MIC_L_OUTPUT+
- net Net-(MK1-OUTPUT-) renamed /MIC_L_OUTPUT-
- net Net-(MK3-OUTPUT+) renamed /MIC_R_OUTPUT+
- net Net-(MK3-OUTPUT-) renamed /MIC_R_OUTPUT-
- net Net-(OA1-IN+) renamed /LT1128CS8_L1_IN+
- net Net-(OA1-OUT) renamed /LT1128CS8_L1_OUT
- net Net-(OA2-IN+) renamed /LT1128CS8_L2_IN+
- net Net-(OA2-OUT) renamed /LT1128CS8_L2_OUT
- net Net-(OA3-IN+) renamed /LT1128CS8_R1_IN+
- net Net-(OA3-OUT) renamed /LT1128CS8_R1_OUT
- net Net-(OA4-IN+) renamed /LT1128CS8_R2_IN+
- net Net-(OA4-OUT) renamed /LT1128CS8_R2_OUT
- C10 pad 1: Net-(OA2-IN-) -> /IN-
- C16 pad 1: Net-(OA3-IN-) -> /IN-
- C19 pad 1: Net-(OA4-IN-) -> /IN-
- C9 pad 1: Net-(OA1-IN-) -> /IN-
- OA1 pad 2: Net-(OA1-IN-) -> /IN-
- OA2 pad 2: Net-(OA2-IN-) -> /IN-
- OA3 pad 2: Net-(OA3-IN-) -> /IN-
- OA4 pad 2: Net-(OA4-IN-) -> /IN-
- R13 pad 1: Net-(OA3-IN-) -> /IN-
- R14 pad 1: Net-(OA4-IN-) -> /IN-
- R6 pad 1: Net-(OA1-IN-) -> /IN-
- R7 pad 1: Net-(OA2-IN-) -> /IN-
Routing:
- added copper zone on F.Cu, net GND
Other:
- board outline added: 100 x 50 mm

Commit message: Update
Parts:
- moved R16 168.8 mm to (88.7, 104.3)
- moved R10 167.1 mm to (95.1, 122.3), turned to 180 degrees
- moved R9 165.7 mm to (98.8, 122.3)
- moved R12 165.1 mm to (91.8, 119.2), turned to -90 degrees
- moved R14 161.5 mm to (84.7, 102.6)
- moved R11 158.2 mm to (101.7, 119.1), turned to 90 degrees
- moved C21 156.2 mm to (84.8, 114.0)
- moved C19 154.8 mm to (84.8, 105.6)
- moved R18 154.2 mm to (87.9, 65.1), turned to 90 degrees
- moved R15 153.2 mm to (112.6, 110.9)
- moved D4 150.5 mm to (219.8, 131.3), turned to 90 degrees
- moved D5 150.3 mm to (219.9, 135.5), turned to 90 degrees
- moved C20 149.3 mm to (92.4, 109.3)
- moved R19 144.8 mm to (96.8, 65.1), turned to 90 degrees
- moved J3 144.6 mm to (92.6, 75.2), turned to -90 degrees
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Connections:
- net /EXT_POWER_12V-_PP renamed /EXT_POWER_12V-
- C10 pad 1: /IN- -> /L2_IN-
- C16 pad 1: /IN- -> /R1_IN-
- C19 pad 1: /IN- -> /R2_IN-
- C9 pad 1: /IN- -> /L1_IN-
- OA1 pad 2: /IN- -> /L1_IN-
- OA2 pad 2: /IN- -> /L2_IN-
- OA3 pad 2: /IN- -> /R1_IN-
- OA4 pad 2: /IN- -> /R2_IN-
- R13 pad 1: /IN- -> /R1_IN-
- R14 pad 1: /IN- -> /R2_IN-
- R6 pad 1: /IN- -> /L1_IN-
- R7 pad 1: /IN- -> /L2_IN-

Commit message: Update
Parts:
- S1: value Switch_WS-SLSU SMT Mini Slide -> 450404015514
- moved C8 23.3 mm to (139.9, 89.0)
- moved OA1 23.3 mm to (141.7, 85.0)
- moved R6 23.3 mm to (136.1, 82.2)
- moved C7 23.3 mm to (147.4, 84.4)
- moved C9 23.3 mm to (136.1, 84.4)
- moved R5 23.3 mm to (142.2, 79.8)
- moved C10 23.2 mm to (157.1, 80.5)
- moved C11 23.2 mm to (165.9, 84.3)
- moved C12 23.2 mm to (158.3, 88.9)
- moved OA2 23.2 mm to (160.0, 84.9)
- moved R7 23.2 mm to (154.2, 84.3)
- moved R8 23.2 mm to (165.9, 86.6)
- moved R14 21.9 mm to (82.8, 124.5), turned to 90 degrees
- moved C19 18.9 mm to (85.1, 124.5), turned to 90 degrees
- moved C21 15.5 mm to (91.1, 128.2), turned to -90 degrees
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Routing:
- added copper zone on B.Cu, net GND
- added copper zone on In1.Cu, net GND
- added copper zone on In2.Cu, net GND

Commit message: Update
Parts:
- removed C10, C9: 470p_C0G, Capacitor_SMD:C_0805_2012Metric
- removed C2, C7, C8: 100n_X7R, Capacitor_SMD:C_0805_2012Metric
- removed C32: 4u7, Capacitor_SMD:C_0805_2012Metric
- removed C39, C41: 47u, Capacitor_SMD:C_0805_2012Metric
- removed C40, C42: 10n_X7R, Capacitor_SMD:C_0805_2012Metric
- removed D1: BZX84C4V3LT1G, Package_TO_SOT_SMD:SOT-23
- removed D3, D6: BZX84C6V2LT1G, Package_TO_SOT_SMD:SOT-23
- removed D4, D5: BZX84C13LT1G, Package_TO_SOT_SMD:SOT-23
- removed J10: JST_XH_2.54_Plug_12V+, Personal_Project:Connector_Power2pin_SHDRRA2W80P0X250_1X2_740X1150X610P
- removed J11: JST_XH_2.54_Plug_12V-, Personal_Project:Connector_Power2pin_SHDRRA2W80P0X250_1X2_740X1150X610P
- removed J12: I2S_Headers, Connector_PinHeader_2.54mm:PinHeader_2x04_P2.54mm_Horizontal
- removed J17: MCLK_Jumper, Connector_PinHeader_2.54mm:PinHeader_1x03_P2.54mm_Vertical
- removed J4: 3V_Selection_Header, Connector_PinHeader_2.54mm:PinHeader_1x03_P2.54mm_Vertical
- removed J9: I/O_Headers, Connector_PinHeader_2.54mm:PinHeader_2x05_P2.54mm_Horizontal
- removed OA1, OA2, OA3, OA4: LT1128CS8, Personal_Project:OpAmp_LT1128CS8_SOIC127P599X175-8N
- removed Q1: MOSFET_SI2333DDS-T1-BE3, Personal_Project:MOSFET_ SI2333DDS_SOT_DS-T1-BE3_VIS
- removed Q3, Q4: MOSFET_SI2343DS-T1-BE3, Personal_Project:MOSFET_ SI2333DDS_SOT_DS-T1-BE3_VIS
- removed R15, R16, R8: 91, Resistor_SMD:R_0805_2012Metric
- removed R18, R19, R2, R26: 100k, Resistor_SMD:R_0805_2012Metric
- removed Z4: Diode_BZX84C6V2-7-F, Personal_Project:Diode_BZX84C6V2_SOT96P240X110-3N
- added ADCD1: ADC_Driver_ADA4940-2ACPZ-R7, Personal_Project:ADC_Driver_ADA4940-2ACPZ-R7_QFN50P400X400X80-25N-D, F.Cu at (151.2, 62.5)
- added FPC1: I2S_FPC_Header, Personal_Project:FPC_SAMTEC_ZF5S-20-01-T-WT, F.Cu at (96.6, 95.2)
- C11, C20: value 100n_X7R -> 10u
- C12, C17, C18: value 100n_X7R -> 100n
- C13: value 2700p_C0G -> 10u
- C14, C5, C6: value 10u -> 100n
- C16, C19: value 470p_C0G -> 10u
- C21: value 100n_X7R -> 2n7
- C22: value 2700p_C0G -> 2n7
- J2: value JST_XH_2.54_Plug_3V3+ -> I2S_OR_LJ_OUT; footprint Personal_Project:Connector_Power2pin_SHDRRA2W80P0X250_1X2_740X1150X610P -> Connector_PinHeader_2.54mm:PinHeader_1x03_P2.54mm_Vertical
- J3: value 3V3_Power_Selector_Jumper -> I/O_Headers_1; footprint Connector_PinHeader_2.54mm:PinHeader_2x03_P2.54mm_Vertical -> Connector_PinHeader_2.54mm:PinHeader_2x05_P2.54mm_Horizontal
- J5: value I/O_Headers -> I/O_Headers_2
- OS1: value Oscillator_ECS-5032MV-122.8-CN-TR -> Oscillator(12.2880MHZ)_ECS-5032MV-122.8-CN-TR
- R1, R10: value 100k -> 200R
- R11, R3: value 10k -> 500R
- R12: value 10k -> 200R
- R13, R14: value 634 -> 22R
- R17: value 22R1 -> 22R
- R4: value 10k -> 22R
- R5: value 91 -> 22R
- R6: value 634 -> 500k
- R7: value 634 -> 200R
- R9: value 100k -> 500k
- S1: value 450404015514 -> Switch_WS-SLSU SMT Mini Slide
- moved C30 147.9 mm to (85.5, 80.8)
- moved LDO1 147.8 mm to (85.8, 77.6)
- moved C31 147.8 mm to (89.9, 76.7)
- moved C36 131.5 mm to (96.3, 77.3), turned to 180 degrees
- moved C35 130.0 mm to (96.5, 71.9), turned to 180 degrees
- moved FB1 127.3 mm to (97.2, 68.9), turned to -90 degrees
- moved C34 126.0 mm to (96.3, 65.8), turned to 180 degrees
- moved C33 123.8 mm to (96.2, 63.5), turned to 180 degrees
- moved J13 122.8 mm to (101.5, 82.4)
- moved J8 108.1 mm to (112.0, 84.5)
- moved J7 96.2 mm to (118.8, 56.5), turned to 90 degrees
- moved C15 96.0 mm to (153.5, 46.9), turned to 180 degrees
- moved J6 94.0 mm to (117.0, 84.6), turned to 90 degrees
- moved R10 88.5 mm to (146.9, 55.3)
- moved C14 84.6 mm to (150.4, 56.0)
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Connections:
- C1 pad 1: +12V -> +5VA
- C11 pad 1: +12V -> +5VA
- C12 pad 1: -12V -> +5VA
- C13 pad 1: /AINL- -> +5VA
- C13 pad 2: /AINL+ -> GND
- C14 pad 1: /LT1128CS8_R1_IN+ -> +5VA
- C14 pad 2: /MIC_R_OUTPUT+ -> GND
- C15 pad 1: /LT1128CS8_R2_IN+ -> /MIC_L_OUTPUT+
- C15 pad 2: /MIC_R_OUTPUT- -> /MIC_L_OUTPUT+_C
- C16 pad 1: /R1_IN- -> /MIC_L_OUTPUT-
- C16 pad 2: /LT1128CS8_R1_OUT -> /MIC_L_OUTPUT-_C
- C17 pad 1: +12V -> +3.3V
- C18 pad 1: -12V -> +3.3V
- C19 pad 1: /R2_IN- -> /MIC_R_OUTPUT+
- C19 pad 2: /LT1128CS8_R2_OUT -> /MIC_R_OUTPUT+_C
- C20 pad 1: +12V -> /MIC_R_OUTPUT-
- C20 pad 2: GND -> /MIC_R_OUTPUT-_C
- C21 pad 1: -12V -> /AINL-
- C21 pad 2: GND -> /AINL+
- C30 pad 1: /LDO_IN -> +5VA
- C31 pad 1: /LD_OUT_3V3 -> +3.3V
- C33 pad 1: /EXT_POWER_5V+_PP -> Net-(Z3-K)
- C34 pad 1: /EXT_POWER_5V+_PP -> Net-(Z3-K)
- C5 pad 1: /LT1128CS8_L1_IN+ -> /VCOM_B_RIGHT
- C5 pad 2: /MIC_L_OUTPUT+ -> GND
- C6 pad 1: /LT1128CS8_L2_IN+ -> /VCOM_B_LEFT
- C6 pad 2: /MIC_L_OUTPUT- -> GND
- FB1 pad 1: /EXT_POWER_5V+_PP -> Net-(Z3-K)
- IC1 pad 4: Net-(IC1-VCC-) -> GND
- J15 pad 1: /VBUS_5V -> /USB_VBUS_5V
- J2 pad 1: GND -> /USB_VBUS_5V
- J2 pad 2: /EXT_POWER_3V3+ -> Net-(J2-Pin_2)
- J3 pad 1: /EXT_POWER_3V3+_PP -> /M0
- J3 pad 2: /EXT_POWER+_NOLDO -> GND
- J3 pad 3: /EXT_POWER_5V+_PP -> /M1
- J3 pad 4: /LDO_IN -> GND
- J3 pad 5: /VBUS_5V -> /MDIV
- J3 pad 6: /LDO_IN -> GND
- LDO1 pad 1: /LDO_IN -> +5VA
- LDO1 pad 3: /LDO_IN -> +5VA
- LDO1 pad 5: /LD_OUT_3V3 -> +3.3V
- R1 pad 1: /MIC_L_OUTPUT+ -> /MIC_L_OUTPUT+_C
- R1 pad 2: GND -> /+IN1
- R10 pad 1: /MIC_R_OUTPUT- -> /MIC_R_OUTPUT+_C
- R10 pad 2: GND -> /+IN2
- R11 pad 1: /LT1128CS8_R1_IN+ -> /-IN2
- R11 pad 2: /VCOM_B_RIGHT -> /+FB2
- R12 pad 1: /VCOM_B_RIGHT -> /MIC_R_OUTPUT-_C
- R12 pad 2: /LT1128CS8_R2_IN+ -> /-IN2
- R13 pad 1: /R1_IN- -> /-OUT2
- R13 pad 2: /AINR+ -> /AINR-
- R14 pad 1: /R2_IN- -> /+OUT2
- R14 pad 2: /AINR- -> /AINR+
- R3 pad 1: /LT1128CS8_L1_IN+ -> /+IN1
- R3 pad 2: /VCOM_B_LEFT -> /-FB1
- R4 pad 1: /VCOM_B_LEFT -> /+OUT1
- R4 pad 2: /LT1128CS8_L2_IN+ -> /AINL+
- R5 pad 1: /LT1128CS8_L1_OUT -> /-OUT1
- R5 pad 2: /AINL+ -> /AINL-
- R6 pad 1: /L1_IN- -> /+FB1
- R6 pad 2: /AINL+ -> /-IN1
- R7 pad 1: /L2_IN- -> /MIC_L_OUTPUT-_C
- R7 pad 2: /AINL- -> /-IN1
- R9 pad 1: /MIC_R_OUTPUT+ -> /+IN2
- R9 pad 2: GND -> /-FB2
- S1 pad 1: /POWER_3V3 -> Net-(Z3-K)
- S1 pad 2: +3.3V -> Net-(J2-Pin_2)
- U1 pad 5: /MCLK -> /MCLK_LOCAL
- Z1 pad 1: /MOSFET_GATE_3V3 -> GND
- Z1 pad 3: /EXT_POWER_3V3+_PP -> /USB_VBUS_5V
- Z3 pad 1: /MOSFET_GATE_12V+ -> GND
- Z3 pad 3: +12V -> Net-(Z3-K)
Routing:
- net +5VA: track 0.00 -> 3.58 mm
- added copper zone on F.Cu, net +5VA
Other:
- board size 100 x 50 mm -> 100 x 56 mm

Commit message: Update
Parts:
- removed ADCD1: ADC_Driver_ADA4940-2ACPZ-R7, Personal_Project:ADC_Driver_ADA4940-2ACPZ-R7_QFN50P400X400X80-25N-D
- removed C25, C37: 1u_X7R, Capacitor_SMD:C_0805_2012Metric
- removed C26, C28, C34, C35, C38: 10n_X7R, Capacitor_SMD:C_0805_2012Metric
- removed C27, C33, C36: 47u, Capacitor_SMD:C_0805_2012Metric
- removed C29: 1uF, Capacitor_SMD:C_0805_2012Metric
- removed C30, C31: 1u, Capacitor_SMD:C_0805_2012Metric
- removed H1, H2, H3, H4: MountingHole_Pad, MountingHole:MountingHole_3.2mm_M3_Pad
- removed IC1: OpAmp_NE5532D, Personal_Project:OpAmp_NE5532DR_SOIC127P600X175-8N
- removed J13: MCLK_DIV_Jumper, Connector_PinHeader_2.54mm:PinHeader_1x03_P2.54mm_Vertical
- removed J14: JST_XH_2.54_Plug_5V+, Personal_Project:Connector_Power2pin_SHDRRA2W80P0X250_1X2_740X1150X610P
- removed J15: USB_B_Micro, Connector_USB:USB_Micro-B_Molex-105017-0001
- removed J16: USB_D_Jumper, Connector_PinHeader_2.54mm:PinHeader_1x02_P2.54mm_Vertical
- removed J2, J6, J7: I2S_OR_LJ_OUT, Connector_PinHeader_2.54mm:PinHeader_1x03_P2.54mm_Vertical
- removed J5: I/O_Headers_2, Connector_PinHeader_2.54mm:PinHeader_2x05_P2.54mm_Horizontal
- removed J8: HP_FILTER_EN, Connector_PinHeader_2.54mm:PinHeader_1x03_P2.54mm_Vertical
- removed MK3: Microphone_ICS-40730, Personal_Project:Microphone_ICS40730
- removed OS1: Oscillator(12.2880MHZ)_ECS-5032MV-122.8-CN-TR, Personal_Project:Oscillator_ECS5032MV250CNTR
- removed R10, R12: 200R, Resistor_SMD:R_0805_2012Metric
- removed R11: 500R, Resistor_SMD:R_0805_2012Metric
- removed R13, R14, R17: 22R, Resistor_SMD:R_0805_2012Metric
- removed R20, R21: 10, Resistor_SMD:R_0805_2012Metric
- removed R22: 5k1, Resistor_SMD:R_0805_2012Metric
- removed R23, R24: 100k, Resistor_SMD:R_0805_2012Metric
- removed R25: 10k, Resistor_SMD:R_0805_2012Metric
- removed S1: Switch_WS-SLSU SMT Mini Slide, Personal_Project:Switch_WS-SLSU SMT Mini Slide
- removed U2: ~, Personal_Project:Button_KMR231GLFS
- removed Z1, Z3: Diode_BZX84C6V2-7-F, Personal_Project:Diode_BZX84C6V2_SOT96P240X110-3N
- added ADCD2: ADC_Driver_ADA4940-2ACPZ-R7, Personal_Project:ADC_Driver_ADA4940-2ACPZ-R7_QFN50P400X400X80-25N-D, F.Cu at (125.3, 53.8)
- added C10: 10u, Capacitor_SMD:C_0805_2012Metric, B.Cu at (108.9, 51.9)
- added C2: 100n, Capacitor_SMD:C_0805_2012Metric, B.Cu at (147.7, 48.3)
- added C32: 10u, Capacitor_SMD:C_0805_2012Metric, B.Cu at (105.6, 52.6)
- added C39: 10u, Capacitor_SMD:C_0805_2012Metric, F.Cu at (123.3, 48.6)
- added C40: 100n, Capacitor_SMD:C_0805_2012Metric, F.Cu at (125.6, 48.6)
- added C41: 10u, Capacitor_SMD:C_0805_2012Metric, F.Cu at (117.1, 55.2)
- added C42: 100n, Capacitor_SMD:C_0805_2012Metric, F.Cu at (119.4, 55.2)
- added C43: 100n, Capacitor_SMD:C_0805_2012Metric, F.Cu at (121.6, 56.2)
- added C44: 100n, Capacitor_SMD:C_0805_2012Metric, F.Cu at (127.2, 58.0)
- added C45: 2n7, Capacitor_SMD:C_0805_2012Metric, F.Cu at (122.8, 63.6)
- added C46: 2n7, Capacitor_SMD:C_0805_2012Metric, F.Cu at (131.9, 63.7)
- added C7: 100n, Capacitor_SMD:C_0805_2012Metric, B.Cu at (110.6, 46.5)
- added C8: 10u, Capacitor_SMD:C_0805_2012Metric, B.Cu at (145.2, 52.9)
- added C9: 10u, Capacitor_SMD:C_0805_2012Metric, B.Cu at (141.9, 52.2)
- added D2: SMAJ6.0A, Personal_Project:DO-214AC-2, F.Cu at (77.5, 72.0)
- added H5: MountingHole_Pad, MountingHole:MountingHole_3.2mm_M3_Pad, F.Cu at (74.0, 54.0)
- added H6: MountingHole_Pad, MountingHole:MountingHole_3.2mm_M3_Pad, F.Cu at (166.0, 54.0)
- added H7: MountingHole_Pad, MountingHole:MountingHole_3.2mm_M3_Pad, F.Cu at (74.0, 96.0)
- added H8: MountingHole_Pad, MountingHole:MountingHole_3.2mm_M3_Pad, F.Cu at (166.0, 96.0)
- added IC2: OpAmp_NE5532D, Personal_Project:OpAmp_NE5532DR_SOIC127P600X175-8N, F.Cu at (108.3, 74.4)
- added J10: HP_FILTER_EN_JMP, Connector_PinHeader_2.54mm:PinHeader_1x03_P2.54mm_Vertical, F.Cu at (151.2, 76.8)
- added J11: MCLK_DIV_JMP, Connector_PinHeader_2.54mm:PinHeader_1x03_P2.54mm_Vertical, F.Cu at (146.3, 76.7)
- added J12: Mode_Selection_Jumpers, Connector_PinHeader_2.54mm:PinHeader_2x03_P2.54mm_Vertical, F.Cu at (140.4, 66.9)
- added J4: I2S_OR_LJ_OUT_JMP, Connector_PinHeader_2.54mm:PinHeader_1x03_P2.54mm_Vertical, F.Cu at (140.3, 76.6)
- added J9: M_OR_S_JMP, Connector_PinHeader_2.54mm:PinHeader_1x03_P2.54mm_Vertical, F.Cu at (109.6, 86.3)
- added JST2: JST_S3B-XH-2.54, Personal_Project:JST_S3B-XH-SHDRRA3W64P0X250_1X3_990X1150X610P, F.Cu at (88.0, 58.5)
- added LDO2: LDO_LDLN050PU33R, Package_DFN_QFN:DFN-8-1EP_3x3mm_P0.65mm_EP1.7x2.05mm, F.Cu at (82.4, 78.3)
- added MK2: Microphone_ICS-40730, Personal_Project:Microphone_ICS40730, B.Cu at (144.0, 47.8)
- added OS2: Oscillator(12.2880MHZ)_ECS-5032MV-122.8-CN-TR, Personal_Project:Oscillator_ECS5032MV250CNTR, F.Cu at (120.5, 90.2)
- added R15: 200R, Resistor_SMD:R_0805_2012Metric, B.Cu at (112.8, 51.9)
- added R16: 200R, Resistor_SMD:R_0805_2012Metric, B.Cu at (108.9, 54.3)
- added R18: 500k, Resistor_SMD:R_0805_2012Metric, B.Cu at (134.9, 51.5)
- added R19: 500k, Resistor_SMD:R_0805_2012Metric, B.Cu at (115.7, 51.1)
- added R2: 200R, Resistor_SMD:R_0805_2012Metric, B.Cu at (141.9, 54.7)
- added R26: 500R, Resistor_SMD:R_0805_2012Metric, B.Cu at (138.0, 54.7)
- added R27: 500R, Resistor_SMD:R_0805_2012Metric, B.Cu at (112.8, 54.3)
- added R28: 22R, Resistor_SMD:R_0805_2012Metric, F.Cu at (123.8, 60.5)
- added R29: 22R, Resistor_SMD:R_0805_2012Metric, F.Cu at (121.6, 60.5)
- added R30: 22R, Resistor_SMD:R_0805_2012Metric, F.Cu at (132.9, 60.6)
- added R31: 22R, Resistor_SMD:R_0805_2012Metric, F.Cu at (130.6, 60.6)
- added R8: 200R, Resistor_SMD:R_0805_2012Metric, B.Cu at (138.0, 52.2)
- added U3: CS5381K-KSZ, Package_SO:SOIC-24W_7.5x15.4mm_P1.27mm, F.Cu at (127.6, 77.0)
- added VS1: VS_STM1813LWX7F, Personal_Project:SOT-23-3_SOT103P237X112-3N, F.Cu at (97.2, 74.0)
- added VS2: VS_STM1818TWX7F, Personal_Project:SOT-23-3_SOT103P237X112-3N, F.Cu at (82.1, 88.2)
- C1: value 100n_X7R -> 1u
- C11, C15: value 10u -> 10n_X7R
- C12, C6: value 100n -> 10n_X7R
- C13: value 10u -> 1u_X7R
- C14, C5: value 100n -> 1u_X7R
- C16: value 10u -> 47u
- C17: value 100n -> 100n_X7R
- C18: value 100n -> 2u2
- C19: value 10u -> 1u
- C20: value 10u -> 2u2
- C21: value 2n7 -> 10n
- C22: value 2n7 -> 100n
- C23: value 1u_X7R -> 4u7
- C24: value 10n_X7R -> 100n
- C3: value 10n_X7R -> 1u_X7R
- C4: value 1u_X7R -> 10n_X7R
- FB1: value BLM21PG601SN1D_0805 -> BLM21AG121BH1D
- FPC1: value I2S_FPC_Header -> FPC_0545481072; footprint Personal_Project:FPC_SAMTEC_ZF5S-20-01-T-WT -> Personal_Project:FPC_0545481072
- J1: value Mode_Selection_Jumpers -> I/O_Headers_2; footprint Connector_PinHeader_2.54mm:PinHeader_2x03_P2.54mm_Vertical -> Connector_PinHeader_2.54mm:PinHeader_2x04_P2.54mm_Horizontal
- J3: footprint Connector_PinHeader_2.54mm:PinHeader_2x05_P2.54mm_Horizontal -> Connector_PinHeader_2.54mm:PinHeader_2x04_P2.54mm_Horizontal
- LDO1: value LDO_TLV75733PDBVR -> LDO_LDLN050PUR; footprint Personal_Project:LDO_SOT95P280X145-5N -> Package_DFN_QFN:DFN-8-1EP_3x3mm_P0.65mm_EP1.7x2.05mm
- MK1: moved to B.Cu
- R1: value 200R -> 10k
- R3: value 500R -> 22R
- R4: value 22R -> 10
- R5: value 22R -> 10R
- R6: value 500k -> 31k6
- R7: value 200R -> 100k
- R9: value 500k -> 10k
- U1: value CS5381 -> SN74LVC1G07DBVR; footprint Package_SO:SOIC-24W_7.5x15.4mm_P1.27mm -> Package_TO_SOT_SMD:SOT-23-5
- moved C1 75.1 mm to (82.3, 74.4), turned to 0 degrees
- moved R7 72.9 mm to (81.9, 62.9), turned to 180 degrees
- moved R6 63.1 mm to (91.8, 70.2), turned to 90 degrees
- moved R9 57.4 mm to (91.8, 66.2), turned to 90 degrees
- moved C17 53.5 mm to (113.5, 73.4)
- moved MK1 52.1 mm to (107.0, 47.7), turned to 90 degrees
- moved C21 50.9 mm to (82.3, 82.2), turned to 180 degrees
- moved C18 47.2 mm to (82.3, 84.6), turned to 0 degrees
- moved C16 44.7 mm to (115.9, 73.3), turned to -90 degrees
- moved C15 44.1 mm to (118.2, 73.3), turned to -90 degrees
- moved C19 43.6 mm to (83.6, 70.0), turned to 90 degrees
- moved J3 43.1 mm to (90.0, 92.4)
- moved J1 38.5 mm to (104.9, 92.4), turned to -90 degrees
- moved C14 38.4 mm to (130.1, 88.5), turned to 0 degrees
- moved C20 36.4 mm to (94.2, 70.2), turned to 90 degrees
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Connections:
- C1 pad 1: +5VA -> /Power_Management/PWR+_PP
- C1 pad 2: Net-(IC1-VCC+) -> GND
- C11 pad 1: +5VA -> /ADC_CS5381K-KSZ/VQ_NE5532D
- C12 pad 1: +5VA -> +3.3V
- C13 pad 1: +5VA -> /ADC_CS5381K-KSZ/VQ_NE5532D
- C14 pad 1: +5VA -> +3.3V
- C15 pad 1: /MIC_L_OUTPUT+ -> /ADC_CS5381K-KSZ/FILT+
- C15 pad 2: /MIC_L_OUTPUT+_C -> GND
- C16 pad 1: /MIC_L_OUTPUT- -> /ADC_CS5381K-KSZ/FILT+
- C16 pad 2: /MIC_L_OUTPUT-_C -> GND
- C17 pad 1: +3.3V -> GND
- C17 pad 2: GND -> +5VA
- C19 pad 1: /MIC_R_OUTPUT+ -> /Power_Management/PWR+_PP
- C19 pad 2: /MIC_R_OUTPUT+_C -> GND
- C20 pad 1: /MIC_R_OUTPUT- -> /Power_Management/OUT_LDLN050PUR
- C20 pad 2: /MIC_R_OUTPUT-_C -> GND
- C21 pad 1: /AINL- -> Net-(LDO2-FB)
- C21 pad 2: /AINL+ -> GND
- C22 pad 1: /AINR- -> /Power_Management/OUT_LDLN050PUR
- C22 pad 2: /AINR+ -> GND
- C23 pad 1: +3.3V -> +5VA
- C24 pad 1: +3.3V -> +5VA
- C3 pad 1: /VQ -> /ADC_CS5381K-KSZ/VDD
- C4 pad 1: /VQ -> /ADC_CS5381K-KSZ/VDD
- C5 pad 1: /VCOM_B_RIGHT -> +3.3V
- C6 pad 1: /VCOM_B_LEFT -> +3.3V
- FB1 pad 1: Net-(Z3-K) -> +5VA
- FB1 pad 2: +5VA -> /Power_Management/OUT_LDLN050PUR
- FPC1 pad 11: /LRCK -> GND
- J1 pad 1: +3.3V -> /ADC_CS5381K-KSZ/~{OVFL}
- J1 pad 2: +3.3V -> GND
- J1 pad 3: /M0 -> /ADC_CS5381K-KSZ/I2S/~{LJ}
- J1 pad 4: /M1 -> GND
- J1 pad 5: GND -> /ADC_CS5381K-KSZ/M/~{S}
- J3 pad 1: /M0 -> /ADC_CS5381K-KSZ/M0
- J3 pad 3: /M1 -> /ADC_CS5381K-KSZ/M1
- J3 pad 5: /MDIV -> /ADC_CS5381K-KSZ/MDIV
- J3 pad 7: /~{DISABLE1}_ADA4940 -> /ADC_CS5381K-KSZ/~{RST}_CS5381
- LDO1 pad 1: +5VA -> /Power_Management/OUT_LDLN050PUR
- LDO1 pad 2: GND -> unconnected-(LDO1-NC-Pad2)
- LDO1 pad 3: +5VA -> Net-(LDO1-FB)
- LDO1 pad 4: unconnected-(LDO1-NC-Pad4) -> GND
- LDO1 pad 5: +3.3V -> /Power_Management/PWR+_PP
- MK1 pad 2: /MIC_L_OUTPUT+ -> /ADC_Driver_ADA4940-2ACPZ-R7/MIC_L_OUT+
- MK1 pad 3: /MIC_L_OUTPUT- -> /ADC_Driver_ADA4940-2ACPZ-R7/MIC_L_OUT-
- Q2 pad 1: /MOSFET_GATE_5V -> /Power_Management/PWR+_GATE
- Q2 pad 2: /EXT_POWER_5V+_PP -> /Power_Management/PWR+_PP
- Q2 pad 3: /EXT_POWER_5V+ -> /Power_Management/PWR+
- R1 pad 1: /MIC_L_OUTPUT+_C -> +3.3V
- R1 pad 2: /+IN1 -> /ADC_CS5381K-KSZ/~{OVFL}
- R3 pad 1: /+IN1 -> /ADC_CS5381K-KSZ/I2S_SDOUT_R
- R3 pad 2: /-FB1 -> /ADC_CS5381K-KSZ/I2S_SDOUT
- R4 pad 1: /+OUT1 -> /ADC_CS5381K-KSZ/VDD
- R4 pad 2: /AINL+ -> +3.3V
- R5 pad 1: /-OUT1 -> /ADC_CS5381K-KSZ/MCLK_R
- R5 pad 2: /AINL- -> /ADC_CS5381K-KSZ/I2S_MCLK_LOCAL
- R6 pad 1: /+FB1 -> /Power_Management/OUT_LDLN050PUR
- R6 pad 2: /-IN1 -> Net-(LDO1-FB)
- R7 pad 1: /MIC_L_OUTPUT-_C -> /Power_Management/PWR+_GATE
- R7 pad 2: /-IN1 -> GND
- R9 pad 1: /+IN2 -> Net-(LDO1-FB)
- R9 pad 2: /-FB2 -> GND
- U1 pad 1: /~{RST} -> unconnected-(U1-NC-Pad1)
- U1 pad 2: /M/~{S} -> /Power_Management/RST_PWR
- U1 pad 3: /LRCK -> GND
- U1 pad 4: /SCLK -> /ADC_CS5381K-KSZ/~{RST}_CS5381
- U1 pad 5: /MCLK_LOCAL -> +3.3V
- Z2 pad 1: /MOSFET_GATE_5V -> /Power_Management/PWR+_GATE
- Z2 pad 3: /EXT_POWER_5V+_PP -> /Power_Management/PWR+_PP
Routing:
- net /ADC_CS5381K-KSZ/VQ_NE5532D: track 0.00 -> 15.4 mm
- net +5VA: track 3.58 -> 0.00 mm
- removed copper zone on F.Cu, net +5VA
Other:
- outline, holes or cut-outs redrawn
- board text added: "MK1"
- board text added: "MK2"

Commit message: Update
Parts:
- added G***: LOGO, Personal_Project:PCB_Logo, F.Cu at (158.3, 63.7)
- C10, C32, C8, C9, R15, R16, R18, R19, R2, R26, R27, R8: moved to F.Cu
- moved J9 49.0 mm to (157.6, 76.5)
- moved MK2 38.5 mm to (105.5, 47.2), turned to 180 degrees
- moved MK1 37.5 mm to (144.5, 47.2), turned to 0 degrees
- moved C2 36.1 mm to (111.7, 45.7), turned to 0 degrees
- moved C7 33.5 mm to (143.8, 50.9), turned to 0 degrees
- moved OS2 14.1 mm to (112.0, 79.0)
- moved C3 14.1 mm to (105.3, 79.0)
- moved C4 14.1 mm to (107.7, 79.0)
- moved J4 13.8 mm to (147.2, 88.6)
- moved J10 13.4 mm to (157.6, 88.6)
- moved R4 13.0 mm to (103.0, 79.0), turned to -90 degrees
- moved VS2 11.1 mm to (92.0, 83.1), turned to 0 degrees
- moved C17 10.3 mm to (110.2, 63.6), turned to 0 degrees
- moved R5 9.49 mm to (117.0, 77.9), turned to 0 degrees
- moved R2 8.70 mm to (134.4, 50.3), turned to 180 degrees
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- renumbered ADCD2 to ADC1
Connections:
- FPC1 pad 4: /Interfaces/I2S1_CK -> /ADC_CS5381K-KSZ/I2S_SCLK
- FPC1 pad 7: /Interfaces/I2S1_WS -> /ADC_CS5381K-KSZ/I2S_LRCK
- FPC1 pad 9: /Interfaces/I2S1_SDI/O -> /ADC_CS5381K-KSZ/I2S_SDOUT
Routing:
- net +5VA: track 0.00 -> 66.0 mm, vias 0 -> 4
- net /ADC_CS5381K-KSZ/M/~{S}: track 0.00 -> 44.9 mm, vias 0 -> 2
- net /ADC_CS5381K-KSZ/~{HPF}: track 0.00 -> 34.9 mm
- net /ADC_Driver_ADA4940-2ACPZ-R7/VCOM_B_RIGHT: track 0.00 -> 32.7 mm
- net /ADC_Driver_ADA4940-2ACPZ-R7/VCOM_B_LEFT: track 0.00 -> 29.0 mm, vias 0 -> 2
- net /ADC_CS5381K-KSZ/M1: track 0.00 -> 25.9 mm
- net /ADC_CS5381K-KSZ/I2S/~{LJ}: track 0.00 -> 21.0 mm
- net +3.3V: track 0.00 -> 20.1 mm
- net /ADC_CS5381K-KSZ/MDIV: track 0.00 -> 17.3 mm
- net /ADC_CS5381K-KSZ/I2S_SCLK: track 0.00 -> 17.2 mm, vias 0 -> 2
- net /Power_Management/PWR+_PP: track 0.00 -> 16.7 mm
- net /ADC_CS5381K-KSZ/I2S_LRCK: track 0.00 -> 15.2 mm, vias 0 -> 2
- net /ADC_CS5381K-KSZ/M0: track 0.00 -> 15.0 mm
- net /ADC_CS5381K-KSZ/I2S_SDOUT: track 0.00 -> 13.6 mm
- net /ADC_CS5381K-KSZ/AINR+: track 0.00 -> 12.1 mm
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- added copper zone on F.Cu, net +3.3V
- added copper zone on F.Cu, net +5VA
- added copper zone on F.Cu, net /ADC_CS5381K-KSZ/FILT+
- added copper zone on F.Cu, net /Power_Management/OUT_LDLN050PUR
- added copper zone on F.Cu, net /Power_Management/PWR+
- added copper zone on F.Cu, net /Power_Management/PWR+_GATE
- added copper zone on F.Cu, net /Power_Management/PWR+_PP

Commit message: Update
Parts:
- removed J1: I/O_Headers_2, Connector_PinHeader_2.54mm:PinHeader_2x04_P2.54mm_Horizontal
- removed J3: I/O_Headers_1, Connector_PinHeader_2.54mm:PinHeader_2x04_P2.54mm_Horizontal
- added J2: I/O_Headers_1, Connector_PinHeader_2.54mm:PinHeader_2x05_P2.54mm_Horizontal, F.Cu at (99.6, 92.0)
- R18, R19: value 500k -> 500R
- moved U1 5.54 mm to (95.5, 83.7)
- moved VS2 1.15 mm to (91.0, 83.7)
Routing:
- net +3.3V: track 20.1 -> 168.2 mm, vias 0 -> 3
- net /ADC_CS5381K-KSZ/~{RST}_CS5381: track 0.00 -> 106.0 mm, vias 0 -> 3
- net /ADC_CS5381K-KSZ/~{OVFL}: track 3.19 -> 59.9 mm, vias 0 -> 1
- net /ADC_CS5381K-KSZ/M0: track 15.0 -> 69.5 mm, vias 0 -> 1
- net /ADC_CS5381K-KSZ/M1: track 25.9 -> 78.9 mm, vias 0 -> 1
- net /ADC_CS5381K-KSZ/~{HPF}: track 34.9 -> 82.8 mm, vias 0 -> 1
- net /Power_Management/RST_PWR: track 0.00 -> 46.5 mm, vias 0 -> 1
- net +5VA: track 66.0 -> 92.6 mm, vias 4 -> 5
- net GND: vias 0 -> 130
Other:
- board text added: "Audio Interface Format"
- board text added: "Div1/Div2"
- board text added: "High Pass Filter"
- board text added: "MCLK Divider"
- board text added: "Master/Slave Mode"
- board text added: "S/M"
