File: ADC_CS5381KKSZ_Board.kicad_pcb (KiCad board)
At the start: 4 copper layers, 100 x 56 mm, 80 parts, among them IC2 OpAmp_NE5532D, J10 HP_FILTER_EN_JMP, J11 MCLK_DIV_JMP, J12 Mode_Selection_Jumpers, J2 I/O_Headers_1, J4 I2S_OR_LJ_OUT_JMP, J9 M_OR_S_JMP, Q2 MOSFET_SI2333DDS-T1-BE3, U1 SN74LVC1G07DBVR, U3 CS5381K-KSZ

Commit message: Update
Parts:
- moved G*** 2.48 mm to (156.6, 61.9)
- moved MK2 0.60 mm to (104.9, 47.2)
- moved MK1 0.54 mm to (145.1, 47.2)
- moved C7 0.50 mm to (144.3, 50.9)
Routing:
- net /ADC_CS5381K-KSZ/~{RST}_CS5381: track 106.0 -> 185.7 mm, vias 3 -> 4
- net +3.3V: track 168.2 -> 239.8 mm, vias 3 -> 6
- net GND: track 11.6 -> 75.7 mm, vias 130 -> 184
- net /ADC_CS5381K-KSZ/AINL-: track 10.9 -> 14.1 mm
- net /ADC_CS5381K-KSZ/AINL+: track 9.00 -> 11.3 mm
- net Net-(LDO1-FB): track 2.67 -> 4.74 mm
- net /ADC_CS5381K-KSZ/M0: track 69.5 -> 70.5 mm
- net /ADC_Driver_ADA4940-2ACPZ-R7/MIC_R_OUT-: track 4.88 -> 5.60 mm
- net /ADC_Driver_ADA4940-2ACPZ-R7/MIC_R_OUT+: track 4.01 -> 4.61 mm
- net /ADC_Driver_ADA4940-2ACPZ-R7/MIC_L_OUT+: track 5.50 -> 6.04 mm
Other:
- board text added: "HPF"
- board text added: "I2S OUT"
- board text added: "M0"
- board text added: "M1"
- board text added: "OVFL"
- board text added: "RST"
- board text removed: "MK1"

Commit message: Update
Parts:
- added G***: LOGO, Personal_Project:PCB_Logo, B.Cu at (130.4, 64.2)
Other:
- board text added: "ADC BOARD Revision: REV B Designer: Peter Hancak ADC DRIVER: ADA4940-2ACPZ-R7 ADC: CS5381K-KSZ LDO: LDLN050PUR, LDLN050PU33R INTERFACE: I2S (FPC) VIN: 2.7 to 6.5V"
- board text added: "VIN:2.7 to 6.5V"

Commit message: Update
Parts:
- removed J2: I/O_Headers_1, Connector_PinHeader_2.54mm:PinHeader_2x05_P2.54mm_Horizontal
- removed R15, R16: 200R, Resistor_SMD:R_0805_2012Metric
- added DI1: Diode_PESD5V0U2BT-Q, Package_TO_SOT_SMD:SOT-23, F.Cu at (108.1, 102.7)
- added DP1: DP_MCP4662-502E_UN, Personal_Project:DP_MCP4662_SOP50P490X110-10N, F.Cu at (143.1, 49.6)
- added DP2: DP_MCP4662-502E_UN, Personal_Project:DP_MCP4662_SOP50P490X110-10N, F.Cu at (118.9, 49.6)
- added J1: DP1_HVC/A0_JMP, Connector_PinHeader_2.54mm:PinHeader_1x03_P2.54mm_Vertical, F.Cu at (98.3, 54.0)
- added J3: DP2_HVC/A0_JMP, Connector_PinHeader_2.54mm:PinHeader_1x03_P2.54mm_Vertical, F.Cu at (102.9, 54.0)
- added J5: I2C1_Headers, Personal_Project:PinHeader_2x03_P2.54mm_Horizontal_Court, F.Cu at (110.8, 92.5)
- added J6: I/O_Headers_1, Connector_PinHeader_2.54mm:PinHeader_2x07_P2.54mm_Horizontal, F.Cu at (99.5, 92.5)
- R18, R26: value 500R -> 1K
- R2, R8: value 200R -> 10k
- moved R8 50.3 mm to (105.6, 89.2)
- moved R2 45.7 mm to (110.5, 89.3)
- moved C7 13.7 mm to (158.0, 51.0)
- moved C8 13.7 mm to (152.0, 50.4)
- moved C9 13.7 mm to (152.0, 48.0)
- moved MK1 13.7 mm to (158.8, 47.3)
- moved G*** 13.1 mm to (118.3, 69.2)
- moved J10 7.47 mm to (164.0, 84.7)
- moved J4 7.46 mm to (153.6, 84.7)
- moved J11 6.92 mm to (153.6, 74.1)
- moved J9 6.92 mm to (164.1, 74.1)
- moved ADC1 6.88 mm to (132.6, 53.7)
- moved C45 6.88 mm to (130.1, 63.5)
- moved R28 6.88 mm to (131.1, 60.4)
- moved C11 6.88 mm to (127.3, 68.7)
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Connections:
- C10 pad 2: /ADC_Driver_ADA4940-2ACPZ-R7/MIC_R_OUT+_C -> /ADC_Driver_ADA4940-2ACPZ-R7/MIC_R_OUT-_C
- C32 pad 2: /ADC_Driver_ADA4940-2ACPZ-R7/MIC_R_OUT-_C -> /ADC_Driver_ADA4940-2ACPZ-R7/MIC_R_OUT+_C
- R2 pad 1: /ADC_Driver_ADA4940-2ACPZ-R7/MIC_L_OUT+_C -> +3.3V
- R2 pad 2: /ADC_Driver_ADA4940-2ACPZ-R7/+IN1 -> /ADC_Driver_ADA4940-2ACPZ-R7/DP1_SDA
- R8 pad 1: /ADC_Driver_ADA4940-2ACPZ-R7/MIC_L_OUT-_C -> +3.3V
- R8 pad 2: /ADC_Driver_ADA4940-2ACPZ-R7/-IN1 -> /ADC_Driver_ADA4940-2ACPZ-R7/DP1_SCL
Routing:
- net GND: track 75.7 -> 87.3 mm, vias 184 -> 191
- net +5VA: track 92.6 -> 103.7 mm
- net /ADC_CS5381K-KSZ/M0: track 70.5 -> 78.0 mm
- net /ADC_CS5381K-KSZ/M1: track 79.3 -> 86.9 mm
- net /ADC_CS5381K-KSZ/~{OVFL}: track 59.9 -> 67.2 mm
- net /ADC_CS5381K-KSZ/~{RST}_CS5381: track 185.7 -> 192.4 mm
- net +3.3V: track 239.8 -> 244.4 mm
- net /ADC_CS5381K-KSZ/I2S_SDOUT: track 13.6 -> 18.1 mm
- net /ADC_CS5381K-KSZ/I2S/~{LJ}: track 21.0 -> 16.7 mm
- net /ADC_CS5381K-KSZ/I2S_LRCK: track 15.2 -> 17.8 mm
- net /ADC_Driver_ADA4940-2ACPZ-R7/+IN2: track 10.4 -> 8.20 mm
- net /ADC_Driver_ADA4940-2ACPZ-R7/+IN1: track 6.92 -> 4.74 mm
- net /ADC_Driver_ADA4940-2ACPZ-R7/-IN2: track 8.51 -> 6.34 mm
- net /ADC_Driver_ADA4940-2ACPZ-R7/-IN1: track 8.86 -> 6.70 mm
- net /ADC_CS5381K-KSZ/M/~{S}: track 44.9 -> 46.5 mm
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Other:
- outline, holes or cut-outs redrawn
- board text added: "ADC BOARD Revision: REV B Designer: Peter Hancak ADC DRIVER: ADA4940-2ACPZ-R7 ADC: CS5381K-KSZ LDO: LDLN050PUR, LDLN050PU33R (Low noise) INTERFACE: I2S (FPC) VIN: 2.7 to 6.5V"
- board text added: "GND"
- board text added: "LOW/HIGH"
- board text added: "Mode"
- board text added: "Mode M1 M0 Output Sample Rate 0 0 2kHz - 50 kHz 0 1 50 kHz - 108 kHz 1 0 100 kHz - 216 khz"
- board text added: "VIN: 5.5 - 6.5V"
- board text removed: "ADC BOARD Revision: REV B Designer: Peter Hancak ADC DRIVER: ADA4940-2ACPZ-R7 ADC: CS5381K-KSZ LDO: LDLN050PUR, LDLN050PU33R INTERFACE: I2S (FPC) VIN: 2.7 to 6.5V"
- board text removed: "VIN:2.7 to 6.5V"

Commit message: Update
Parts:
- FPC1: value FPC_0545481072 -> FPC_10051922-1010ELF; footprint Personal_Project:FPC_0545481072 -> Personal_Project:FPC_10051922_1010
- moved FPC1 50.0 mm to (164.2, 126.6), turned to 180 degrees
- moved C43 50.0 mm to (166.7, 88.9)
- moved C3 50.0 mm to (152.1, 109.0)
- moved C45 50.0 mm to (170.1, 93.5)
- moved C8 50.0 mm to (192.0, 80.4)
- moved FB1 50.0 mm to (140.0, 101.6)
- moved G*** 50.0 mm to (158.3, 99.2)
- moved IC2 50.0 mm to (155.3, 97.7)
- moved J1 50.0 mm to (138.3, 84.0)
- moved J5 50.0 mm to (150.8, 122.5)
- moved MK1 50.0 mm to (198.8, 77.3)
- moved MK2 50.0 mm to (144.6, 77.2)
- moved R19 50.0 mm to (165.5, 77.4)
- moved R26 50.0 mm to (178.3, 81.0)
- moved R8 50.0 mm to (145.6, 119.2)
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Routing:
- net GND: track 87.3 -> 97.1 mm

Commit message: Update
Parts:
- removed ADC1: ADC_Driver_ADA4940-2ACPZ-R7, Personal_Project:ADC_Driver_ADA4940-2ACPZ-R7_QFN50P400X400X80-25N-D
- removed DI1: Diode_PESD5V0U2BT-Q, Package_TO_SOT_SMD:SOT-23
- removed DP1, DP2: DP_MCP4662-502E_UN, Personal_Project:DP_MCP4662_SOP50P490X110-10N
- removed J1: DP1_HVC/A0_JMP, Connector_PinHeader_2.54mm:PinHeader_1x03_P2.54mm_Vertical
- removed J3: DP2_HVC/A0_JMP, Connector_PinHeader_2.54mm:PinHeader_1x03_P2.54mm_Vertical
- removed J5: I2C1_Headers, Personal_Project:PinHeader_2x03_P2.54mm_Horizontal_Court
- removed R2, R8: 10k, Resistor_SMD:R_0805_2012Metric
- added AMP1: ADC_Driver_ADA4940-2ACPZ-R7, Personal_Project:ADC_Driver_ADA4940-2ACPZ-R7_QFN50P400X400X80-25N-D, F.Cu at (172.6, 83.7)
- added R10: 2K, Resistor_SMD:R_0805_2012Metric, F.Cu at (182.7, 80.5)
- added R11: 2K, Resistor_SMD:R_0805_2012Metric, F.Cu at (182.7, 78.2)
- added R12: 2K, Resistor_SMD:R_0805_2012Metric, F.Cu at (162.4, 78.1)
- added R13: 2K, Resistor_SMD:R_0805_2012Metric, F.Cu at (162.4, 80.5)
- R18, R26: value 1K -> 1K_RN73H2ATTD1001B25
- R19, R27: value 500R -> 1K_RN73H2ATTD1001B25
- moved G*** 5.81 mm to (158.6, 93.4)
- moved C7 1.95 mm to (199.9, 81.0)
- moved MK1 1.95 mm to (200.7, 77.3)
- moved C8 1.88 mm to (193.8, 80.5)
- moved C9 1.88 mm to (193.8, 78.1)
- moved R26 1.35 mm to (179.6, 81.2)
- moved R18 1.34 mm to (179.6, 77.4)
Connections:
- C10 pad 2: /ADC_Driver_ADA4940-2ACPZ-R7/MIC_R_OUT-_C -> /ADC_Driver_ADA4940-2ACPZ-R7/MIC_R_C_OUT+
- C32 pad 2: /ADC_Driver_ADA4940-2ACPZ-R7/MIC_R_OUT+_C -> /ADC_Driver_ADA4940-2ACPZ-R7/MIC_R_C_OUT-
- C8 pad 2: /ADC_Driver_ADA4940-2ACPZ-R7/MIC_L_OUT+_C -> /ADC_Driver_ADA4940-2ACPZ-R7/MIC_L_C_OUT+
- C9 pad 2: /ADC_Driver_ADA4940-2ACPZ-R7/MIC_L_OUT-_C -> /ADC_Driver_ADA4940-2ACPZ-R7/MIC_L_C_OUT-
- J6 pad 11: /ADC_Driver_ADA4940-2ACPZ-R7/DP1_HVC/A0 -> /ADC_Driver_ADA4940-2ACPZ-R7/~{DISABLE1}_ADA4940
- J6 pad 13: /ADC_Driver_ADA4940-2ACPZ-R7/DP2_HVC/A0 -> /ADC_Driver_ADA4940-2ACPZ-R7/~{DISABLE2}_ADA4940
Routing:
- net /ADC_Driver_ADA4940-2ACPZ-R7/MIC_L_C_OUT+: track 0.00 -> 9.90 mm
- net /ADC_Driver_ADA4940-2ACPZ-R7/MIC_R_C_OUT-: track 0.00 -> 9.90 mm
- net /ADC_Driver_ADA4940-2ACPZ-R7/MIC_L_C_OUT-: track 0.00 -> 9.89 mm
- net /ADC_Driver_ADA4940-2ACPZ-R7/MIC_R_C_OUT+: track 0.00 -> 9.87 mm
- net +5VA: track 103.7 -> 106.9 mm
- net /ADC_Driver_ADA4940-2ACPZ-R7/+IN2: track 8.20 -> 10.4 mm
- net /ADC_Driver_ADA4940-2ACPZ-R7/-IN2: track 6.34 -> 8.50 mm
- net /ADC_Driver_ADA4940-2ACPZ-R7/MIC_L_OUT-_C: track 2.05 -> 0.00 mm
- net /ADC_Driver_ADA4940-2ACPZ-R7/MIC_L_OUT+_C: track 2.04 -> 0.00 mm
- net /ADC_Driver_ADA4940-2ACPZ-R7/MIC_R_OUT-_C: track 1.99 -> 0.00 mm
- net +3.3V: track 244.4 -> 246.4 mm
- net /ADC_Driver_ADA4940-2ACPZ-R7/MIC_R_OUT+_C: track 1.94 -> 0.00 mm
- net GND: track 97.1 -> 95.5 mm, vias 191 -> 211
- net /ADC_Driver_ADA4940-2ACPZ-R7/+IN1: track 4.74 -> 6.34 mm
- net /ADC_Driver_ADA4940-2ACPZ-R7/-IN1: track 6.70 -> 8.20 mm
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Other:
- board text added: "DIS1"
- board text added: "DIS2"
- board text added: "Notes: ~{DISABLE}_ADA4940 Pins are active LOW (Disabled) - Disable ADA4940 when the device is not being used - Has internal pull-up ADA4940 Rg and Rf should be metal film R Rg around 2k Ohms"
- board text added: "Rg"

Commit message: Update
Parts:
- R30, R31: value 22R -> 22R_Metal_Film
- moved C2 1.27 mm to (150.6, 76.6), turned to -90 degrees
- moved MK2 0.69 mm to (143.9, 77.2)
- moved C17 0.27 mm to (156.8, 93.6)
- moved C10 0.24 mm to (151.2, 78.1)
- moved C32 0.24 mm to (151.3, 80.5)
Routing:
- net +3.3V: track 246.4 -> 86.0 mm, vias 6 -> 7
- net /ADC_Driver_ADA4940-2ACPZ-R7/~{DISABLE1}_ADA4940: track 0.00 -> 116.6 mm, vias 0 -> 3
- net /ADC_Driver_ADA4940-2ACPZ-R7/~{DISABLE2}_ADA4940: track 0.00 -> 105.7 mm, vias 0 -> 3
- net /ADC_CS5381K-KSZ/~{RST}_CS5381: track 192.4 -> 87.7 mm, vias 4 -> 3
- net +5VA: track 106.9 -> 30.1 mm, vias 5 -> 11
- net GND: track 95.5 -> 124.3 mm, vias 211 -> 363
- net /ADC_CS5381K-KSZ/AINL+: track 11.3 -> 19.7 mm
- net /ADC_CS5381K-KSZ/AINR-: track 11.7 -> 19.7 mm
- net /ADC_CS5381K-KSZ/AINR+: track 12.1 -> 20.0 mm
- net /ADC_CS5381K-KSZ/VDD: track 7.84 -> 0.27 mm
- net /Power_Management/PWR+_PP: track 16.7 -> 12.2 mm
- net /ADC_CS5381K-KSZ/~{HPF}: track 84.4 -> 80.9 mm
- net /ADC_Driver_ADA4940-2ACPZ-R7/+OUT2: track 5.26 -> 8.35 mm
- net /ADC_Driver_ADA4940-2ACPZ-R7/-OUT2: track 3.94 -> 6.68 mm
- net /ADC_Driver_ADA4940-2ACPZ-R7/+IN1: track 6.34 -> 8.61 mm
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- added copper zone on B.Cu, net +3.3V
- added copper zone on B.Cu, net +5VA
- added copper zone on F.Cu, net /ADC_CS5381K-KSZ/VDD

Commit message: Update
Parts:
- added R2: 22R, Resistor_SMD:R_0603_1608Metric, F.Cu at (168.4, 116.6)
- added R8: 22R, Resistor_SMD:R_0603_1608Metric, F.Cu at (179.9, 116.9)
- R3, R5: footprint Resistor_SMD:R_0805_2012Metric -> Resistor_SMD:R_0603_1608Metric
- moved R3 9.73 mm to (170.2, 116.6)
Connections:
- R3 pad 1: /ADC_CS5381K-KSZ/I2S_SDOUT_R -> /ADC_CS5381K-KSZ/I2S_SCLK_R
- R3 pad 2: /ADC_CS5381K-KSZ/I2S_SDOUT -> /ADC_CS5381K-KSZ/I2S_SCLK
- U3 pad 3: /ADC_CS5381K-KSZ/I2S_LRCK -> /ADC_CS5381K-KSZ/I2S_LRCK_R
- U3 pad 4: /ADC_CS5381K-KSZ/I2S_SCLK -> /ADC_CS5381K-KSZ/I2S_SCLK_R
Routing:
- net GND: track 124.3 -> 98.6 mm, vias 363 -> 436
- net /ADC_CS5381K-KSZ/I2S_LRCK: track 17.8 -> 23.5 mm, vias 2 -> 0
- net /ADC_CS5381K-KSZ/I2S_SCLK: track 18.1 -> 23.7 mm, vias 2 -> 0
- net /ADC_CS5381K-KSZ/I2S_LRCK_R: track 0.00 -> 4.76 mm
- net /ADC_CS5381K-KSZ/I2S_SCLK_R: track 0.00 -> 4.51 mm
- net /ADC_CS5381K-KSZ/I2S_SDOUT: track 20.1 -> 22.1 mm
- net +5VA: track 30.1 -> 30.9 mm

Commit message: Update
Parts:
- removed C32: 10u, Capacitor_SMD:C_0805_2012Metric
- added C25: 10u, Capacitor_SMD:C_1812_4532Metric, F.Cu at (152.2, 81.3)
- added R14: 10k, Resistor_SMD:R_0805_2012Metric, F.Cu at (156.2, 102.8)
- C10, C8, C9: footprint Capacitor_SMD:C_0805_2012Metric -> Capacitor_SMD:C_1812_4532Metric
- C39, C41, C43, C44: footprint Capacitor_SMD:C_0805_2012Metric -> Capacitor_SMD:C_0603_1608Metric
- C40, C42: value 100n -> 1n; footprint Capacitor_SMD:C_0805_2012Metric -> Capacitor_SMD:C_0603_1608Metric
- R18, R19, R26, R27: value 1K_RN73H2ATTD1001B25 -> 1k
- moved R30 3.25 mm to (176.9, 90.4)
- moved R18 2.90 mm to (176.8, 78.2), turned to 0 degrees
- moved R19 2.83 mm to (168.2, 78.2), turned to 0 degrees
- moved C44 2.57 mm to (173.3, 90.2), turned to -90 degrees
- moved C43 1.75 mm to (165.4, 87.7), turned to 180 degrees
- moved C9 1.44 mm to (192.7, 77.2)
- moved C8 1.41 mm to (192.7, 81.3)
- moved C10 1.36 mm to (152.2, 77.2)
- moved R31 1.26 mm to (179.1, 90.4)
- moved C46 1.07 mm to (178.1, 93.4), turned to 0 degrees
- moved C42 0.55 mm to (166.1, 85.1)
- moved C39 0.52 mm to (172.5, 77.0)
- moved C7 0.26 mm to (200.2, 81.0)
- moved MK1 0.26 mm to (201.0, 77.3)
- moved C40 0.12 mm to (172.5, 78.8)
Connections:
- net /ADC_Driver_ADA4940-2ACPZ-R7/+OUT1 renamed /ADC_Driver_ADA4940-2ACPZ-R7/OUT1+
- net /ADC_Driver_ADA4940-2ACPZ-R7/+OUT2 renamed /ADC_Driver_ADA4940-2ACPZ-R7/OUT2+
- net /ADC_Driver_ADA4940-2ACPZ-R7/-OUT1 renamed /ADC_Driver_ADA4940-2ACPZ-R7/OUT1-
- net /ADC_Driver_ADA4940-2ACPZ-R7/-OUT2 renamed /ADC_Driver_ADA4940-2ACPZ-R7/OUT2-
Routing:
- net /ADC_CS5381K-KSZ/AINR+: track 20.0 -> 2.29 mm
- net /ADC_CS5381K-KSZ/AINR-: track 19.7 -> 2.21 mm
- net /ADC_CS5381K-KSZ/AINL+: track 19.7 -> 2.32 mm
- net /ADC_CS5381K-KSZ/AINL-: track 13.6 -> 2.56 mm, vias 2 -> 0
- net GND: track 98.6 -> 93.6 mm, vias 436 -> 444
- net /ADC_Driver_ADA4940-2ACPZ-R7/-FB2: track 10.1 -> 5.37 mm
- net /ADC_Driver_ADA4940-2ACPZ-R7/+FB1: track 10.1 -> 5.46 mm
- net /ADC_Driver_ADA4940-2ACPZ-R7/MIC_R_OUT+: track 5.06 -> 8.24 mm
- net /ADC_Driver_ADA4940-2ACPZ-R7/OUT2+: track 8.35 -> 5.29 mm
- net /ADC_Driver_ADA4940-2ACPZ-R7/OUT1-: track 8.46 -> 6.44 mm
- net /ADC_Driver_ADA4940-2ACPZ-R7/MIC_L_C_OUT+: track 10.1 -> 8.23 mm
- net /ADC_Driver_ADA4940-2ACPZ-R7/MIC_R_C_OUT+: track 10.1 -> 8.24 mm
- net /ADC_Driver_ADA4940-2ACPZ-R7/MIC_L_OUT-: track 5.09 -> 6.93 mm
- net /ADC_Driver_ADA4940-2ACPZ-R7/MIC_L_C_OUT-: track 10.1 -> 8.33 mm
- net /ADC_Driver_ADA4940-2ACPZ-R7/OUT2-: track 6.68 -> 4.91 mm
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