File: ADC_CS5381KKSZ_Board.kicad_pcb (KiCad board)
At the start: 4 copper layers, 100 x 56 mm, 84 parts, among them IC2 OpAmp_NE5532D, J10 HP_FILTER_EN_JMP, J11 MCLK_DIV_JMP, J12 Mode_Selection_Jumpers, J4 I2S_OR_LJ_OUT_JMP, J6 I/O_Headers_1, J9 M_OR_S_JMP, Q2 MOSFET_SI2333DDS-T1-BE3, U1 SN74LVC1G07DBVR, U3 CS5381K-KSZ

Commit message: Update Readme
Routing:
- net /ADC_CS5381K-KSZ/AINR+: track 2.29 -> 12.4 mm
- net /ADC_CS5381K-KSZ/AINR-: track 2.21 -> 12.3 mm
- net /ADC_CS5381K-KSZ/AINL+: track 2.32 -> 12.3 mm
- net /ADC_CS5381K-KSZ/AINL-: track 2.56 -> 12.5 mm

Commit message: Update
Parts:
- C22, C23, C24, FB1: moved to B.Cu
- moved C22 29.6 mm to (167.2, 101.6)
- moved C23 27.1 mm to (165.9, 98.4), turned to 0 degrees
- moved C24 27.1 mm to (165.9, 95.9), turned to 0 degrees
- moved FB1 24.8 mm to (164.8, 101.6)
