File: Power_Management.kicad_sch (KiCad schematic)
At the start: 17 parts, among them IC2 OpAmp_NE5532D, J13 I2S_OR_LJ_OUT, J8 JST_XH_2.54_Plug_5V+, Q2 MOSFET_SI2333DDS-T1-BE3

Commit message: Update
Connections:
- net VQ renamed VQ_NE5532D
Changed lines of the file:
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@@
+	)
+	(junction
+		(at 101.6 166.37)
+		(diameter 0)
+		(color 0 0 0 0)
 	)
 	(junction
@@
 	(wire
 		(pts
+			(xy 101.6 166.37) (xy 119.38 166.37)
+		)
+		(stroke
+			(width 0)
+			(type default)
+		)
+	)
+	(wire
+		(pts
 			(xy 99.06 45.72) (xy 138.43 45.72)
 		)
@@
 	(wire
 		(pts
-			(xy 97.79 166.37) (xy 119.38 166.37)
+			(xy 97.79 166.37) (xy 101.6 166.37)
 		)
 		(stroke
@@
 	(wire
 		(pts
+			(xy 53.34 163.83) (xy 53.34 176.53)
+		)
+		(stroke
+			(width 0)
+			(type default)
+		)
+	)
+	(wire
+		(pts
 			(xy 106.68 55.88) (xy 116.84 55.88)
 		)
@@
 	(wire
 		(pts
+			(xy 101.6 166.37) (xy 101.6 176.53)
+		)
+		(stroke
+			(width 0)
+			(type default)
+		)
+	)
+	(wire
+		(pts
 			(xy 187.96 132.08) (xy 187.96 134.62)
 		)
@@
 		(pts
 			(xy 224.79 55.88) (xy 224.79 58.42)
+		)
+		(stroke
+			(width 0)
+			(type default)
+		)
+	)
+	(wire
+		(pts
+			(xy 53.34 176.53) (xy 101.6 176.53)
 		)
 		(stroke
@@
 		)
 	)
-	(label "VQ"
+	(label "VQ_NE5532D"
 		(at 119.38 166.37 180)
 		(fields_autoplaced yes)
@@
 		)
 	)
-	(label "VQ"
+	(label "VQ_NE5532D"
 		(at 53.34 163.83 0)
 		(fields_autoplaced yes)
@@
 		)
 	)
+	(hierarchical_label "VCOM_B_RIGHT"
+		(shape bidirectional)
+		(at 119.38 161.29 0)
+		(fields_autoplaced yes)
+		(effects
+			(font
+				(size 1.27 1.27)
+			)
+			(justify left)
+		)
+	)
+	(hierarchical_label "VQ_NE5532D"
+		(shape bidirectional)
+		(at 119.38 166.37 0)
+		(fields_autoplaced yes)
+		(effects
+			(font
+				(size 1.27 1.27)
+			)
+			(justify left)
+		)
+	)
+	(hierarchical_label "VCOM_B_LEFT"
+		(shape bidirectional)
+		(at 53.34 158.75 180)
+		(fields_autoplaced yes)
+		(effects
+			(font
+				(size 1.27 1.27)
+			)
+			(justify right)
+		)
+	)

Commit message: Update
Parts:
- removed C21, C24: 47u, Capacitor_SMD:C_0805_2012Metric, symbol Device:C_Polarized
- removed C22, C23: 10n_X7R, Capacitor_SMD:C_0805_2012Metric, symbol Device:C
- removed FB1: BLM21PG601SN1D_0805, Capacitor_SMD:C_0805_2012Metric, symbol Device:FerriteBead
- removed J13: I2S_OR_LJ_OUT, Connector_PinHeader_2.54mm:PinHeader_1x03_P2.54mm_Vertical, symbol Connector_Generic:Conn_01x03
- removed J8: JST_XH_2.54_Plug_5V+, Personal_Project:Connector_Power2pin_SHDRRA2W80P0X250_1X2_740X1150X610P, symbol Personal_Projects:Connector_Power2pin_JST_XH_2.54_Plug
- removed LDO2: LDO_TLV75733PDBVR, Personal_Project:LDO_SOT95P280X145-5N, symbol Personal_Projects:LDO_TLV75733PDBVR
- removed Q2: MOSFET_SI2333DDS-T1-BE3, Personal_Project:MOSFET_ SI2333DDS_SOT_DS-T1-BE3_VIS, symbol Personal_Projects:MOSFET_SI2333DDS-T1-BE3
- removed R7: 100k, Resistor_SMD:R_0805_2012Metric, symbol Device:R
- removed S1: Switch_WS-SLSU SMT Mini Slide, Personal_Project:Switch_WS-SLSU SMT Mini Slide, symbol Personal_Projects:Switch_WS-SLSU SMT Mini Slide
- removed Z2, Z3: Diode_BZX84C6V2-7-F, Personal_Project:Diode_BZX84C6V2_SOT96P240X110-3N, symbol Personal_Projects:Diode_BZX84C6V2-7-F
- added C19: 1u, Capacitor_SMD:C_0805_2012Metric, symbol Device:C
- added C20: 2u2, Capacitor_SMD:C_0805_2012Metric, symbol Device:C
- added C25, C27: 10u, Capacitor_SMD:C_0805_2012Metric, symbol Device:C
- added C30: 470n, Capacitor_SMD:C_0805_2012Metric, symbol Device:C
- added C33, C36: 47u, Capacitor_SMD:C_0805_2012Metric, symbol Device:C_Polarized
- added C34, C35: 10n_X7R, Capacitor_SMD:C_0805_2012Metric, symbol Device:C
- added D1: SMAJ6.0A, Personal_Project:DO-214AC-2, symbol Personal_Projects:DIODE_SMAJ6.0A
- added FB2: BLM21PG601SN1D_0805, Capacitor_SMD:C_0805_2012Metric, symbol Device:FerriteBead
- added J1: JST_XH_2.54_Plug_5V+, Personal_Project:Connector_Power2pin_SHDRRA2W80P0X250_1X2_740X1150X610P, symbol Personal_Projects:Connector_Power2pin_JST_XH_2.54_Plug
- added J3: I2S_OR_LJ_OUT, Connector_PinHeader_2.54mm:PinHeader_1x03_P2.54mm_Vertical, symbol Connector_Generic:Conn_01x03
- added LDO1: LDO_LDLN050PUR, Package_DFN_QFN:DFN-8-1EP_3x3mm_P0.65mm_EP1.7x2.05mm, symbol Personal_Projects:LDO_LDLN050PUR
- added LDO2: LDO_LDLN050PU33R, Package_DFN_QFN:DFN-8-1EP_3x3mm_P0.65mm_EP1.7x2.05mm, symbol Personal_Projects:LDO_LDLN050PUR
- added LDO3: LDO_LD39200PU33R, Package_DFN_QFN:DFN-6-1EP_3x3mm_P0.95mm_EP1.7x2.6mm, symbol Personal_Projects:LDO_LD39200PU33R
- added Q1: MOSFET_SI2333DDS-T1-BE3, Personal_Project:MOSFET_ SI2333DDS_SOT_DS-T1-BE3_VIS, symbol Personal_Projects:MOSFET_SI2333DDS-T1-BE3
- added R10, R6: 31k6, Resistor_SMD:R_0805_2012Metric, symbol Device:R
- added R11, R14, R9: 10k, Resistor_SMD:R_0805_2012Metric, symbol Device:R
- added R12: 100k, Resistor_SMD:R_0805_2012Metric, symbol Device:R
- added R13: 90k, Resistor_SMD:R_0805_2012Metric, symbol Device:R
- added S2: Switch_WS-SLSU SMT Mini Slide, Personal_Project:Switch_WS-SLSU SMT Mini Slide, symbol Personal_Projects:Switch_WS-SLSU SMT Mini Slide
- added Z1: Diode_BZX84C6V2-7-F, Personal_Project:Diode_BZX84C6V2_SOT96P240X110-3N, symbol Personal_Projects:Diode_BZX84C6V2-7-F
- C18: value 1u -> 2u2
Connections:
- net +3.3V: now also C27.1, C30.1, LDO2.1 (OUT), LDO3.1 (OUT), R10.1, R13.2
- net +5VA: now also C35.1, C36.1, FB2.2; no longer C1.1
- net EXT_POWER_5V+: now also J1.2 (POWER+), Q1.3 (D)
- net EXT_POWER_5V+_PP: now also J3.3 (Pin_3), Q1.2 (S), Z1.3 (K)
- net GND: now also C19.2, C20.2, C25.2, C27.2, C33.2, C34.2, C35.2, C36.2, D1.2 (A), J1.1 (POWER-), LDO1.4 (GND_1), LDO1.9 (GND_2), LDO2.4 (GND_1), LDO2.9 (GND_2), LDO3.3 (GND), LDO3.7 (EPAD), R11.2, R12.2, R14.1, R9.2
- net MOSFET_GATE_5V: now also Q1.1 (G), R12.1, Z1.1 (A)
- net USB_VBUS_5V: now also J3.1 (Pin_1)
- new net: LDO1.3 (FB), R6.2, R9.1
- new net: J3.2 (Pin_2), S2.2
- new net: C30.2, LDO3.2 (ADJ/SENSE), R13.1, R14.2
- new net: LDO2.3 (FB), R10.2, R11.1
- new net EN: LDO3.5 (EN)
- new net OUT_LD39200DPUR: C20.1, C25.1, C33.1, C34.1, FB2.1, LDO1.1 (OUT), LDO3.6 (IN), R6.1
- new net PG: LDO3.4 (PG)
- new net VIN_LDLN050PUR: C1.1, C19.1, D1.1 (K), LDO1.5 (EN), LDO1.8 (IN), LDO2.5 (EN), LDO2.8 (IN), S2.1
- no-connect marks 5 -> 11
Other:
- note added: "Protects the MAX 6V VIN"
- note added: "To LDO_LD39200PU33R 3V3 LDO"
- note added: "VIN from 1.25 V to 6.0 V"
- note added: "VIN: 2.7 V to 6.5 V"
- note added: "VOUT​=1.208⋅(1+31600/10000)≈5.0253 V"
- note removed: "If shutdown capability is not required, connect EN to IN."
- moved on the sheet: C17, IC2

Commit message: Update
Parts:
- removed J3: I2S_OR_LJ_OUT, Connector_PinHeader_2.54mm:PinHeader_1x03_P2.54mm_Vertical, symbol Connector_Generic:Conn_01x03
- removed R10: 31k6, Resistor_SMD:R_0805_2012Metric, symbol Device:R
- removed R11: 10k, Resistor_SMD:R_0805_2012Metric, symbol Device:R
- added C21: 10n, Capacitor_SMD:C_0805_2012Metric, symbol Device:C
- added VS1: VS_STM1813LWX7F, Personal_Project:SOT-23-3_SOT103P237X112-3N, symbol Personal_Projects:VS_STM1813LWX7F
- added VS2: VS_STM1818TWX7F, Personal_Project:SOT-23-3_SOT103P237X112-3N, symbol Personal_Projects:VS_STM1813LWX7F
Connections:
- net +3.3V: now also VS2.2 (VCC)
- net EXT_POWER_5V+_PP: now also S2.2
- net GND: now also C21.2, VS1.3 (VSS), VS2.3 (VSS)
- net OUT_LD39200DPUR: no longer C20.1, C33.1, C34.1, FB2.1, LDO1.1 (OUT), R6.1
- net at LDO2.3 (FB): now also C21.1
- new net OUT_LDLN050PUR: C20.1, C33.1, C34.1, FB2.1, LDO1.1 (OUT), R6.1, VS1.2 (VCC)
- new net RST_STM1813LWX7F: VS1.1 (~{RST})
- new net RST_STM1818TWX7F: VS2.1 (~{RST})
Other:
- note removed: "To LDO_LD39200PU33R 3V3 LDO"
- moved on the sheet: C33, C34, C35, C36, FB2

Commit message: Update
Parts:
- removed J1: JST_XH_2.54_Plug_5V+, Personal_Project:Connector_Power2pin_SHDRRA2W80P0X250_1X2_740X1150X610P, symbol Personal_Projects:Connector_Power2pin_JST_XH_2.54_Plug
- added JST1: JST_S3B-XH-2.54, Personal_Project:JST_S3B-XH-SHDRRA3W64P0X250_1X3_990X1150X610P, symbol Personal_Projects:JST_S3B-XH-A-1_LF_SN
Connections:
- net RST_STM1818TWX7F is gone; now on net *RST: VS2.1 (~{RST})
- net GND: now also JST1.2 (PWR-)
- net EXT_POWER_5V+ renamed PWR+
- net PWR+: now also JST1.1 (PWR+)
- net RST_STM1813LWX7F renamed *RST
- net *RST: now also JST1.3 (RST)
Other:
- note removed: "Input voltage range: 5V (Exact)"

Commit message: Update
Parts:
- removed C25, C27: 10u, Capacitor_SMD:C_0805_2012Metric, symbol Device:C
- removed C30: 470n, Capacitor_SMD:C_0805_2012Metric, symbol Device:C
- removed D1: SMAJ6.0A, Personal_Project:DO-214AC-2, symbol Personal_Projects:DIODE_SMAJ6.0A
- removed JST1: JST_S3B-XH-2.54, Personal_Project:JST_S3B-XH-SHDRRA3W64P0X250_1X3_990X1150X610P, symbol Personal_Projects:JST_S3B-XH-A-1_LF_SN
- removed LDO3: LDO_LD39200PU33R, Package_DFN_QFN:DFN-6-1EP_3x3mm_P0.95mm_EP1.7x2.6mm, symbol Personal_Projects:LDO_LD39200PU33R
- removed Q1: MOSFET_SI2333DDS-T1-BE3, Personal_Project:MOSFET_ SI2333DDS_SOT_DS-T1-BE3_VIS, symbol Personal_Projects:MOSFET_SI2333DDS-T1-BE3
- removed R12: 100k, Resistor_SMD:R_0805_2012Metric, symbol Device:R
- removed R13: 90k, Resistor_SMD:R_0805_2012Metric, symbol Device:R
- removed R14: 10k, Resistor_SMD:R_0805_2012Metric, symbol Device:R
- removed S2: Switch_WS-SLSU SMT Mini Slide, Personal_Project:Switch_WS-SLSU SMT Mini Slide, symbol Personal_Projects:Switch_WS-SLSU SMT Mini Slide
- removed Z1: Diode_BZX84C6V2-7-F, Personal_Project:Diode_BZX84C6V2_SOT96P240X110-3N, symbol Personal_Projects:Diode_BZX84C6V2-7-F
- added D2: SMAJ6.0A, Personal_Project:DO-214AC-2, symbol Personal_Projects:DIODE_SMAJ6.0A
- added JST2: JST_S3B-XH-2.54, Personal_Project:JST_S3B-XH-SHDRRA3W64P0X250_1X3_990X1150X610P, symbol Personal_Projects:JST_S3B-XH-A-1_LF_SN
- added Q2: MOSFET_SI2333DDS-T1-BE3, Personal_Project:MOSFET_ SI2333DDS_SOT_DS-T1-BE3_VIS, symbol Personal_Projects:MOSFET_SI2333DDS-T1-BE3
- added R7: 100k, Resistor_SMD:R_0805_2012Metric, symbol Device:R
- added U1: SN74LVC1G07DBVR, Package_TO_SOT_SMD:SOT-23-5, symbol 74xGxx:74LVC1G07
- added Z2: Diode_BZX84C6V2-7-F, Personal_Project:Diode_BZX84C6V2_SOT96P240X110-3N, symbol Personal_Projects:Diode_BZX84C6V2-7-F
Connections:
- net *RST: now also U1.4
- net +3.3V: now also U1.5 (VCC)
- net GND: now also D2.2 (A), JST2.2 (PWR-), R7.2, U1.3 (GND)
- net PWR+: now also JST2.1 (PWR+), Q2.3 (D)
- net VIN_LDLN050PUR renamed PWR+_PP
- net PWR+_PP: now also D2.1 (K), Q2.2 (S), Z2.3 (K)
- new net PWR+_GATE: Q2.1 (G), R7.1, Z2.1 (A)
- new net RST_PWR: JST2.3 (RST), U1.2
- no-connect marks 11 -> 7
Other:
- note added: "NO PU"
- note removed: "ON/OFF Switch"
- note removed: "Pin 2 connects to one or three"
- note removed: "VIN from 1.25 V to 6.0 V"
- moved on the sheet: C1, C17, C18, C21, IC2, LDO2, VS2

Commit message: Update
Parts:
- removed C33, C36: 47u, Capacitor_SMD:C_0805_2012Metric, symbol Device:C_Polarized
- removed C34, C35: 10n_X7R, Capacitor_SMD:C_0805_2012Metric, symbol Device:C
- removed FB2: BLM21PG601SN1D_0805, Capacitor_SMD:C_0805_2012Metric, symbol Device:FerriteBead
- added C22, C24: 100n, Capacitor_SMD:C_0805_2012Metric, symbol Device:C
- added C23: 4u7, Capacitor_SMD:C_0805_2012Metric, symbol Device:C
- added FB1: BLM21AG121BH1D, Capacitor_SMD:C_0805_2012Metric, symbol Device:FerriteBead
Connections:
- net +5VA: now also C23.1, C24.1, FB1.1
- net GND: now also C22.2, C23.2, C24.2
- net OUT_LDLN050PUR: now also C22.1, FB1.2
Other:
- note added: "120Ohm@100MHz"
- note removed: "To generate 3V3"

Commit message: Update
Connections:
- net +5VA: now also C17.2, IC2.8 (VCC+); no longer C17.1
- net GND: now also C17.1
- net VCOM_B_LEFT: now also IC2.6 (2IN-), IC2.7 (2OUT); no longer IC2.1 (1OUT), IC2.2 (1IN-)
- net VCOM_B_RIGHT: now also IC2.1 (1OUT), IC2.2 (1IN-); no longer IC2.6 (2IN-), IC2.7 (2OUT)
Other:
- moved on the sheet: C17
