File: Power_Management.kicad_sch (KiCad schematic)
At the start: 23 parts, among them IC2 OpAmp_NE5532D, Q2 MOSFET_SI2333DDS-T1-BE3, U1 SN74LVC1G07DBVR

Commit message: Update
Other:
- note added: "(5k5 INT PU)"
- note added: "REQUIRES PU"
- note removed: "NO PU"
- moved on the sheet: VS2
Changed lines of the file:
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@@
 	(wire
 		(pts
-			(xy 175.26 124.46) (xy 152.4 124.46)
+			(xy 154.94 124.46) (xy 152.4 124.46)
 		)
 		(stroke
@@
 	(wire
 		(pts
-			(xy 200.66 127) (xy 200.66 124.46)
+			(xy 180.34 127) (xy 180.34 124.46)
 		)
 		(stroke
@@
 	(wire
 		(pts
-			(xy 200.66 124.46) (xy 198.12 124.46)
+			(xy 180.34 124.46) (xy 177.8 124.46)
 		)
 		(stroke
@@
 	(wire
 		(pts
-			(xy 139.7 121.92) (xy 175.26 121.92)
+			(xy 139.7 121.92) (xy 154.94 121.92)
 		)
 		(stroke
@@
 		(pts
 			(xy 212.09 87.63) (xy 227.33 87.63)
+		)
+		(stroke
+			(width 0)
+			(type default)
+		)
+	)
+	(polyline
+		(pts
+			(xy 242.57 102.87) (xy 254 102.87)
 		)
 		(stroke
@@
 		)
 	)
+	(text "REQUIRES PU"
+		(exclude_from_sim no)
+		(at 207.518 155.702 0)
+		(effects
+			(font
+				(size 1 1)
+			)
+		)
+	)
 	(text "Protects the MAX 6V VIN"
 		(exclude_from_sim no)
@@
 		)
 	)
-	(text "NO PU"
-		(exclude_from_sim no)
-		(at 172.974 125.984 0)
+	(text "VIN: 2.7 V to 6.5 V"
+		(exclude_from_sim no)
+		(at 59.436 124.46 0)
 		(effects
 			(font
@@
 		)
 	)
-	(text "VIN: 2.7 V to 6.5 V"
-		(exclude_from_sim no)
-		(at 59.436 124.46 0)
+	(text "VOUT​=1.208⋅(1+31600/10000)≈5.0253 V"
+		(exclude_from_sim no)
+		(at 97.028 110.998 0)
 		(effects
 			(font
@@
 		)
 	)
-	(text "VOUT​=1.208⋅(1+31600/10000)≈5.0253 V"
-		(exclude_from_sim no)
-		(at 97.028 110.998 0)
+	(text "(5k5 INT PU)"
+		(exclude_from_sim no)
+		(at 162.306 128.778 0)
 		(effects
 			(font
@@
 		)
 	)
-	(text "NO PU"
-		(exclude_from_sim no)
-		(at 143.51 105.918 0)
+	(text "(5k5 INT PU)"
+		(exclude_from_sim no)
+		(at 145.542 105.918 0)
 		(effects
 			(font
@@
 	(symbol
 		(lib_id "power:GND")
-		(at 200.66 127 0)
+		(at 180.34 127 0)
 		(mirror y)
 		(unit 1)
@@
 		(dnp no)
 		(property "Reference" "#PWR031"
-			(at 200.66 133.35 0)
+			(at 180.34 133.35 0)
 			(effects
 				(font
@@
 		)
 		(property "Value" "GND"
-			(at 203.2 130.048 90)
+			(at 182.88 130.048 90)
 			(effects
 				(font
@@
 		)
 		(property "Footprint" ""
-			(at 200.66 127 0)
+			(at 180.34 127 0)
 			(effects
 				(font
@@
 		)
 		(property "Datasheet" ""
-			(at 200.66 127 0)
+			(at 180.34 127 0)
 			(effects
 				(font
@@
 		)
 		(property "Description" "Power symbol creates a global label with name \"GND\" , ground"
-			(at 200.66 127 0)
+			(at 180.34 127 0)
 			(effects
 				(font
@@
 	(symbol
 		(lib_id "Personal_Projects:VS_STM1813LWX7F")
-		(at 175.26 124.46 0)
+		(at 154.94 124.46 0)
 		(mirror x)
 		(unit 1)
@@
 		(dnp no)
 		(property "Reference" "VS2"
-			(at 180.086 114.808 0)
+			(at 159.766 114.808 0)
 			(effects
 				(font
@@
 		)
 		(property "Value" "VS_STM1818TWX7F"
-			(at 187.198 117.094 0)
+			(at 166.878 117.094 0)
 			(effects
 				(font
@@
 		)
 		(property "Footprint" "Personal_Project:SOT-23-3_SOT103P237X112-3N"
-			(at 199.39 29.54 0)
+			(at 179.07 29.54 0)
 			(effects
 				(font
@@
 		)
 		(property "Datasheet" "https://componentsearchengine.com/Datasheets/1/STM1813LWX7F.pdf"
-			(at 199.39 -70.46 0)
+			(at 179.07 -70.46 0)
 			(effects
 				(font
@@
 		)
 		(property "Description" "STM1813LWX7F, Reset Monitor 3 V, 3.3 V, 5 V Active Low, Open Drain, reset 3-Pin SOT-23"
-			(at 175.26 114.3 0)
+			(at 154.94 114.3 0)
 			(effects
 				(font
@@
 		)
 		(property "Height" "1.12"
-			(at 199.39 -270.46 0)
+			(at 179.07 -270.46 0)
 			(effects
 				(font
@@
 		)
 		(property "Mouser Part Number" "511-STM1813LWX7F"
-			(at 199.39 -370.46 0)
+			(at 179.07 -370.46 0)
 			(effects
 				(font
@@
 		)
 		(property "Mouser Price/Stock" ""
-			(at 199.39 -470.46 0)
+			(at 179.07 -470.46 0)
 			(effects
 				(font
@@
 		)
 		(property "Manufacturer_Name" "STMicroelectronics"
-			(at 199.39 -570.46 0)
+			(at 179.07 -570.46 0)
 			(effects
 				(font
@@
 		)
 		(property "Manufacturer_Part_Number" "STM1813LWX7F"
-			(at 199.39 -670.46 0)
-			(effects
-				(font
+			(at 179.07 -670.46 0)
+			(effects
+				(font
