File: Power_Management.kicad_sch (KiCad schematic)
At the start: 23 parts, among them IC2 OpAmp_NE5532D, Q2 MOSFET_SI2333DDS-T1-BE3, U1 SN74LVC1G07DBVR

Commit message: Update
Other:
- note added: "5V Quiet LDO: LT3042EMSE#PBF (LT3042EMSE(TOKMAS) cheap version) -2.5V LDO: LT3094EMSE#TRPBF /and charge pump TC7660SEOA (+5V to -5V) Microphone 3.3V LDO: TPS7A2033 (source from quiet LT3042 5V) Architecture: two single channel op-amps Voltage: +3.6V to -1.8V LM27762DSSR POWER TOPOLOGY: ┌───> 5.0V to CS5381 VA (Analog 5V Rail) ~55mA │ [LT3042 5.0V Rail] ──┼───> [TPS7A2033] ──> 3.3V to ICS-40720 Mi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"
