File: Interfaces.kicad_sch (KiCad schematic)
At the start: 11 parts, among them J1 USB_D_Jumper, J2 I/O_Headers_1, J3 USB_B_Micro, J7 I/O_Headers_2

Commit message: Update
Parts:
- removed J1: USB_D_Jumper, Connector_PinHeader_2.54mm:PinHeader_1x02_P2.54mm_Vertical, symbol Connector_Generic:Conn_01x02
- removed J3: USB_B_Micro, Connector_USB:USB_Micro-B_Molex-105017-0001, symbol Connector:USB_B_Micro
- removed R6: 100k, Resistor_SMD:R_0805_2012Metric, symbol Device:R
- removed Z4: Diode_BZX84C6V2-7-F, Personal_Project:Diode_BZX84C6V2_SOT96P240X110-3N, symbol Personal_Projects:Diode_BZX84C6V2-7-F
Connections:
- net I2S/~{LJ} renamed I2S/~{LJ}
- net M/~{S} renamed M/~{S}
Other:
- note removed: "Leave D lines floating for 500mA Short data lines for 1000mA"

Commit message: Update
Parts:
- removed J2: I/O_Headers_1, Connector_PinHeader_2.54mm:PinHeader_2x05_P2.54mm_Horizontal, symbol Connector_Generic:Conn_02x05_Odd_Even
- removed J7: I/O_Headers_2, Connector_PinHeader_2.54mm:PinHeader_2x05_P2.54mm_Horizontal, symbol Connector_Generic:Conn_02x05_Odd_Even
- added J1: I/O_Headers_2, Connector_PinHeader_2.54mm:PinHeader_2x04_P2.54mm_Vertical, symbol Connector_Generic:Conn_02x04_Odd_Even
- added J3: I/O_Headers_1, Connector_PinHeader_2.54mm:PinHeader_2x04_P2.54mm_Vertical, symbol Connector_Generic:Conn_02x04_Odd_Even
Connections:
- net GND: now also J1.2 (Pin_2), J1.4 (Pin_4), J1.6 (Pin_6), J1.8 (Pin_8), J3.2 (Pin_2), J3.4 (Pin_4), J3.6 (Pin_6), J3.8 (Pin_8)
- net I2S/~{LJ}: now also J1.3 (Pin_3)
- net M0: now also J3.1 (Pin_1)
- net M1: now also J3.3 (Pin_3)
- net MDIV: now also J3.5 (Pin_5)
- net M/~{S}: now also J1.5 (Pin_5)
- net ~{HPF}: now also J1.7 (Pin_7)
- net ~{OVFL}: now also J1.1 (Pin_1)
- new net *RST: J3.7 (Pin_7)

Commit message: Update
Parts:
- removed FPC2: I2S_FPC_Header, Personal_Project:FPC_SAMTEC_ZF5S-20-01-T-WT, symbol Personal_Projects:FPC_ZF5S-20-01-T-WT
- added FPC1: FPC_0545481072, Personal_Project:FPC_0545481072, symbol Personal_Projects:FPC_0545481072
Connections:
- net GND: now also FPC1.1, FPC1.10, FPC1.11 (MP1), FPC1.12 (MP2), FPC1.3, FPC1.5, FPC1.6, FPC1.8
- new net I2S1_CK: FPC1.4
- new net I2S1_MCK: FPC1.2
- new net I2S1_SDI/O: FPC1.9
- new net I2S1_WS: FPC1.7
Other:
- moved on the sheet: J1, J3

Commit message: Update
Parts:
- J1, J3: footprint Connector_PinHeader_2.54mm:PinHeader_2x04_P2.54mm_Vertical -> Connector_PinHeader_2.54mm:PinHeader_2x04_P2.54mm_Horizontal
Changed lines of the file:
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@@
 			)
 		)
-		(property "Footprint" "Connector_PinHeader_2.54mm:PinHeader_2x04_P2.54mm_Vertical"
+		(property "Footprint" "Connector_PinHeader_2.54mm:PinHeader_2x04_P2.54mm_Horizontal"
 			(at 99.06 96.52 0)
 			(effects
@@
 			)
 		)
-		(property "Footprint" "Connector_PinHeader_2.54mm:PinHeader_2x04_P2.54mm_Vertical"
+		(property "Footprint" "Connector_PinHeader_2.54mm:PinHeader_2x04_P2.54mm_Horizontal"
 			(at 99.06 62.23 0)
 			(effects

Commit message: Update
Parts:
- removed J1: I/O_Headers_2, Connector_PinHeader_2.54mm:PinHeader_2x04_P2.54mm_Horizontal, symbol Connector_Generic:Conn_02x04_Odd_Even
- removed J3: I/O_Headers_1, Connector_PinHeader_2.54mm:PinHeader_2x04_P2.54mm_Horizontal, symbol Connector_Generic:Conn_02x04_Odd_Even
- added J2: I/O_Headers_1, Connector_PinHeader_2.54mm:PinHeader_2x05_P2.54mm_Horizontal, symbol Connector_Generic:Conn_02x05_Odd_Even
Connections:
- net *RST: now also J2.9 (Pin_9)
- net GND: now also J2.10 (Pin_10), J2.2 (Pin_2), J2.4 (Pin_4), J2.6 (Pin_6), J2.8 (Pin_8)
- net M0: now also J2.3 (Pin_3)
- net M1: now also J2.5 (Pin_5)
- net ~{HPF}: now also J2.1 (Pin_1)
- net ~{OVFL}: now also J2.7 (Pin_7)

Commit message: Update
Parts:
- removed J2: I/O_Headers_1, Connector_PinHeader_2.54mm:PinHeader_2x05_P2.54mm_Horizontal, symbol Connector_Generic:Conn_02x05_Odd_Even
- added DI1: Diode_PESD5V0U2BT-Q, Package_TO_SOT_SMD:SOT-23, symbol Personal_Projects:Diode_PESD5V0U2BT-Q
- added J5: I2C1_Headers, Personal_Project:PinHeader_2x03_P2.54mm_Horizontal_Court, symbol Connector_Generic:Conn_02x03_Odd_Even
- added J6: I/O_Headers_1, Connector_PinHeader_2.54mm:PinHeader_2x07_P2.54mm_Horizontal, symbol Connector_Generic:Conn_02x07_Odd_Even
- added R2, R8: 10k, Resistor_SMD:R_0805_2012Metric, symbol Device:R
Connections:
- net *RST: now also J6.9 (Pin_9)
- net GND: now also DI1.3 (CC), J5.2 (Pin_2), J5.3 (Pin_3), J5.4 (Pin_4), J5.6 (Pin_6), J6.10 (Pin_10), J6.12 (Pin_12), J6.14 (Pin_14), J6.2 (Pin_2), J6.4 (Pin_4), J6.6 (Pin_6), J6.8 (Pin_8)
- net M0: now also J6.3 (Pin_3)
- net M1: now also J6.5 (Pin_5)
- net ~{HPF}: now also J6.1 (Pin_1)
- net ~{OVFL}: now also J6.7 (Pin_7)
- new net +3.3V: R2.1, R8.1
- new net DP1_HVC/A0: J6.11 (Pin_11)
- new net DP2_HVC/A0: J6.13 (Pin_13)
- new net I2C_SCL_HDR: DI1.2 (K2), J5.5 (Pin_5), R8.2
- new net I2C_SDA_HDR: DI1.1 (K1), J5.1 (Pin_1), R2.2
Other:
- note added: "Place ESD close to the header"
- note removed: "Disable Pins Active LOW"
- moved on the sheet: FPC1, H5, H6, H7, H8

Commit message: Update
Parts:
- removed FPC1: FPC_0545481072, Personal_Project:FPC_0545481072, symbol Personal_Projects:FPC_0545481072
- added FPC1: FPC_10051922-1010ELF, Personal_Project:FPC_10051922_1010, symbol Personal_Projects:FPC_10051922-1010ELF
Connections:
- net GND: now also FPC1.1, FPC1.10, FPC1.11 (MP1), FPC1.12 (MP2), FPC1.3, FPC1.5, FPC1.6, FPC1.8
- net I2S1_CK: now also FPC1.4
- net I2S1_MCK: now also FPC1.2
- net I2S1_SDI/O: now also FPC1.9
- net I2S1_WS: now also FPC1.7
Changed lines of the file:
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@@
 	)
 	(symbol
-		(lib_id "Personal_Projects:FPC_0545481072")
+		(lib_id "Personal_Projects:FPC_10051922-1010ELF")
 		(at 172.72 52.07 0)
 		(unit 1)
@@
 		(dnp no)
 		(property "Reference" "FPC1"
-			(at 172.72 42.672 0)
+			(at 184.15 35.814 0)
 			(effects
 				(font
-					(size 1.27 1.27)
+					(size 1.524 1.524)
 				)
 				(justify right)
 			)
 		)
-		(property "Value" "FPC_0545481072"
-			(at 172.72 45.212 0)
+		(property "Value" "FPC_10051922-1010ELF"
+			(at 207.01 38.608 0)
 			(effects
 				(font
-					(size 1.27 1.27)
+					(size 1.524 1.524)
 				)
 				(justify right)
 			)
 		)
-		(property "Footprint" "Personal_Project:FPC_0545481072"
-			(at 194.31 146.99 0)
+		(property "Footprint" "Personal_Project:FPC_10051922_1010"
+			(at 172.72 99.06 0)
 			(effects
 				(font
 					(size 1.27 1.27)
+					(italic yes)
 				)
-				(justify left top)
 				(hide yes)
 			)
 		)
-		(property "Datasheet" "https://www.molex.com/en-us/products/part-detail-pdf/545481072?display=pdf"
-			(at 194.31 246.99 0)
+		(property "Datasheet" "10051922-1010ELF"
+			(at 172.72 95.25 0)
 			(effects
 				(font
 					(size 1.27 1.27)
+					(italic yes)
 				)
-				(justify left top)
 				(hide yes)
 			)
 		)
-		(property "Description" "0.50mm Pitch Easy-On FFC/FPC Connector, 1.20mm Height, Right-Angle, Surface Mount, ZIF, Bottom Contact Style, 10 Circuits, Gold (Au) Plating"
-			(at 172.72 82.55 0)
+		(property "Description" ""
+			(at 185.42 52.07 0)
 			(effects
 				(font
@@
 			)
 		)
-		(property "Height" "1.3"
-			(at 194.31 446.99 0)
-			(effects
-				(font
-					(size 1.27 1.27)
-				)
-				(justify left top)
-				(hide yes)
-			)
+		(pin "6"
 		)
-		(property "Arrow Part Number" "0545481072"
-			(at 194.31 546.99 0)
-			(effects
-				(font
-					(size 1.27 1.27)
-				)
-				(justify left top)
-				(hide yes)
-			)
-		)
-		(property "Arrow Price/Stock" ""
-			(at 194.31 646.99 0)
-			(effects
-				(font
-					(size 1.27 1.27)
-				)
-				(justify left top)
-				(hide yes)
-			)
-		)
-		(property "Manufacturer_Name" "Molex"
-			(at 194.31 746.99 0)
-			(effects
-				(font
-					(size 1.27 1.27)
-				)
-				(justify left top)
-				(hide yes)
-			)
-		)
-		(property "Manufacturer_Part_Number" "0545481072"
-			(at 194.31 846.99 0)
-			(effects
-				(font
-					(size 1.27 1.27)
-				)
-				(justify left top)
-				(hide yes)
-			)
+		(pin "9"
 		)
 		(pin "4"
@@
 		(pin "7"
 		)
-		(pin "6"
+		(pin "2"
 		)
 		(pin "5"
 		)
-		(pin "2"
+		(pin "3"
 		)
 		(pin "8"
 		)
-		(pin "3"
+		(pin "12"
 		)
 		(pin "10"
 		)
-		(pin "12"
+		(pin "1"
 		)
 		(pin "11"
 		)
-		(pin "9"
-		)
-		(pin "1"
-		)
 		(instances

Commit message: Update
Parts:
- removed DI1: Diode_PESD5V0U2BT-Q, Package_TO_SOT_SMD:SOT-23, symbol Personal_Projects:Diode_PESD5V0U2BT-Q
- removed J5: I2C1_Headers, Personal_Project:PinHeader_2x03_P2.54mm_Horizontal_Court, symbol Connector_Generic:Conn_02x03_Odd_Even
- removed R2, R8: 10k, Resistor_SMD:R_0805_2012Metric, symbol Device:R
Connections:
- net DP1_HVC/A0 renamed ~{DISABLE1}_ADA4940
- net DP2_HVC/A0 renamed ~{DISABLE2}_ADA4940
Other:
- note removed: "Place ESD close to the header"
