File: ADC_Driver_ADA4940-2ACPZ-R7.kicad_sch (KiCad schematic)
At the start: 29 parts

Commit message: Update
Other:
- note added: "DISABLE is asserted by applying a low logic level"
Changed lines of the file:
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@@
+		)
+	)
+	(text "DISABLE is asserted by applying a low logic level"
+		(exclude_from_sim no)
+		(at 162.56 54.61 0)
+		(effects
+			(font
+				(size 1 1)
+			)
+			(justify left)
 		)
 	)

Commit message: Update
Parts:
- renumbered MK2 to MK1, MK4 to MK2
Changed lines of the file:
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@@
-		)
-	)
-	(label "-VS2_1"
-		(at 186.69 92.71 0)
-		(fields_autoplaced yes)
-		(effects
-			(font
-				(size 1.27 1.27)
-			)
-			(justify left bottom)
 		)
 	)
@@
 			)
 			(justify right bottom)
-		)
-	)
-	(label "-VS2_2"
-		(at 186.69 90.17 0)
-		(fields_autoplaced yes)
-		(effects
-			(font
-				(size 1.27 1.27)
-			)
-			(justify left bottom)
 		)
 	)
@@
 		(dnp no)
 		(fields_autoplaced yes)
-		(property "Reference" "MK4"
+		(property "Reference" "MK2"
 			(at 45.72 107.95 0)
 			(effects
@@
 			(project "ADC_CS5381KKSZ_Board"
 				(path "/532b720a-d345-4e8b-bed0-e606731588e9/e34874d5-b551-4e69-8606-4abb22c39edc"
-					(reference "MK4")
+					(reference "MK2")
 					(unit 1)
 				)
@@
 		(dnp no)
 		(fields_autoplaced yes)
-		(property "Reference" "MK2"
+		(property "Reference" "MK1"
 			(at 44.45 60.96 0)
 			(effects
@@
 			(project "ADC_CS5381KKSZ_Board"
 				(path "/532b720a-d345-4e8b-bed0-e606731588e9/e34874d5-b551-4e69-8606-4abb22c39edc"
-					(reference "MK2")
-					(unit 1)
-				)
+					(reference "MK1")
+					(unit 1)
+				)

Commit message: Update
Parts:
- R18, R19: value 500k -> 500R
- renumbered ADCD2 to ADC1
Changed lines of the file:
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@@
 			)
 		)
-		(property "Value" "500k"
+		(property "Value" "500R"
 			(at 115.57 77.978 90)
 			(effects
@@
 		(dnp no)
 		(fields_autoplaced yes)
-		(property "Reference" "ADCD2"
+		(property "Reference" "ADC1"
 			(at 177.8 78.7714 0)
 			(effects
@@
 			(project "ADC_CS5381KKSZ_Board"
 				(path "/532b720a-d345-4e8b-bed0-e606731588e9/e34874d5-b551-4e69-8606-4abb22c39edc"
-					(reference "ADCD2")
+					(reference "ADC1")
 					(unit 1)
 				)
@@
 			)
 		)
-		(property "Value" "500k"
+		(property "Value" "500R"
 			(at 115.57 99.314 90)
 			(effects

Commit message: Update
Parts:
- removed R15, R16, R2, R8: 200R, Resistor_SMD:R_0805_2012Metric, symbol Device:R
- added DP1, DP2: DP_MCP4662-502E_UN, Personal_Project:DP_MCP4662_SOP50P490X110-10N, symbol Personal_Projects:DP_MCP4662-502E_UN
- added J1: DP1_HVC/A0_JMP, Connector_PinHeader_2.54mm:PinHeader_1x03_P2.54mm_Vertical, symbol Connector_Generic:Conn_01x03
- added J3: DP2_HVC/A0_JMP, Connector_PinHeader_2.54mm:PinHeader_1x03_P2.54mm_Vertical, symbol Connector_Generic:Conn_01x03
- R18, R26: value 500R -> 1K
Connections:
- net +3.3V: now also DP1.10 (VDD), DP2.10 (VDD), DP2.9 (A1), J1.1 (Pin_1), J3.1 (Pin_1)
- net +IN1: now also DP1.7 (P0W)
- net +IN2: now also DP2.6 (P1W)
- net -IN1: now also DP1.6 (P1W)
- net -IN2: now also DP2.7 (P0W)
- net GND: now also DP1.4 (VSS), DP1.9 (A1), DP2.4 (VSS), J1.3 (Pin_3), J3.3 (Pin_3)
- net MIC_L_OUT+_C: now also DP1.8 (P0B)
- net MIC_L_OUT-_C: now also DP1.5 (P1B)
- net MIC_R_OUT+_C: now also C32.2, DP2.5 (P1B); no longer C10.2
- net MIC_R_OUT-_C: now also C10.2, DP2.8 (P0B); no longer C32.2
- new net DP1_HVC/A0: DP1.1 (HVC/A0), J1.2 (Pin_2)
- new net DP1_SCL: DP1.2 (SCL)
- new net DP1_SDA: DP1.3 (SDA)
- new net DP2_HVC/A0: DP2.1 (HVC/A0), J3.2 (Pin_2)
- new net DP2_SCL: DP2.2 (SCL)
- new net DP2_SDA: DP2.3 (SDA)
Other:
- note added: "Pins A0 and A1 are latched at start. The A0 pin is then used to alllow EEPROM write"
- note added: "The two resistors set the open loop gain G = 2.5 Per leg RFB = 500 Ohm RG = 200 Ohm"
- note removed: "The two resistors set the open loop gain G = 2.5 Per leg"
- moved on the sheet: ADC1, C10, C2, C32, C39, C40, C41, C42, C43, C44, C45, C46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

Commit message: Update
Parts:
- R19, R27: value 500R -> 1K
Other:
- note added: "2. Dielectric Absorption (Ceramic Capacitor Distortions) This is where the "special" capacitor conversation actually matters. If you use cheap X7R or Z5U ceramic capacitors in the signal path, they change their capacitance as the voltage changes. This creates a non-linear distortion that can sound like graininess or crackling during loud bass notes. The Fix: For any capacitor actually touching th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"
Changed lines of the file:
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@@
 		)
 	)
+	(text "2. Dielectric Absorption (Ceramic Capacitor Distortions)\n\nThis is where the \"special\" capacitor conversation actually matters. If you use cheap X7R or Z5U ceramic capacitors in the signal path, they change their capacitance as the voltage changes. This creates a non-linear distortion that can sound like graininess or crackling during loud bass notes.\n\nThe Fix: For any capacitor actually touching the audio signal, use Film capacitors (Polypropylene is king) or C0G/NP0 ceramics. These are stable and won't \"color\" or crackle the sound.\n\nResistors\n2. Choosing the Right Material (The \"Crackle\" Factor)\n\nNot all resistors are made the same. The material inside matters for audio:\n\nCarbon Composition (Avoid): These are the old-school brown cylinders. They are \"noisy\" and have high Voltage Coefficient of Resistance. As the audio signal voltage changes, the resistance changes slightly, which creates a grainy, crackling distortion.\n\nThick Film Surface Mount (Standard): These are okay for general electronics, but they can still be slightly noisy for sensitive audio.\n\nThin Film / Metal Film (Recommended): These are the gold standard for audio. They have very low noise and high stability. If you are using surface-mount parts, look for \"Thin Film\" resistors."
+		(exclude_from_sim no)
+		(at 183.896 37.338 0)
+		(effects
+			(font
+				(size 1.27 1.27)
+				(thickness 0.254)
+				(bold yes)
+			)
+		)
+	)
 	(text "It is also possible to connect the VOCM input to a \ncommon-mode level (CML) output of an ADC. However, \ncare must be taken to ensure that the output has \nsufficient drive capability. The input impedance of \nthe VOCM pin is approximately 250 kΩ."
 		(exclude_from_sim no)
@@
 				)
 				(justify left)
-				(hide yes)
 			)
 		)
@@
 			)
 		)
-		(property "Value" "500R"
+		(property "Value" "1K"
 			(at 153.924 124.46 90)
 			(effects
@@
 			)
 		)
-		(property "Value" "500R"
+		(property "Value" "1K"
 			(at 132.08 101.854 90)
 			(effects

Commit message: Update
Parts:
- removed DP1, DP2: DP_MCP4662-502E_UN, Personal_Project:DP_MCP4662_SOP50P490X110-10N, symbol Personal_Projects:DP_MCP4662-502E_UN
- removed J1: DP1_HVC/A0_JMP, Connector_PinHeader_2.54mm:PinHeader_1x03_P2.54mm_Vertical, symbol Connector_Generic:Conn_01x03
- removed J3: DP2_HVC/A0_JMP, Connector_PinHeader_2.54mm:PinHeader_1x03_P2.54mm_Vertical, symbol Connector_Generic:Conn_01x03
- added R10, R11, R12, R13: 2K, Resistor_SMD:R_0805_2012Metric, symbol Device:R
- R18, R19, R26, R27: value 1K -> 1K_RN73H2ATTD1001B25
- R30, R31: value 22R -> 22R_Metal_Film
- renumbered ADC1 to AMP1
Connections:
- net +IN1: now also R10.2
- net +IN2: now also R12.2
- net -IN1: now also R11.2
- net -IN2: now also R13.2
- net MIC_L_OUT+_C renamed MIC_L_C_OUT+
- net MIC_L_C_OUT+: now also R10.1
- net MIC_L_OUT-_C renamed MIC_L_C_OUT-
- net MIC_L_C_OUT-: now also R11.1
- net MIC_R_OUT+_C renamed MIC_R_C_OUT-
- net MIC_R_C_OUT-: now also R13.1
- net MIC_R_OUT-_C renamed MIC_R_C_OUT+
- net MIC_R_C_OUT+: now also R12.1
Other:
- note added: "Film Capacitors (PPS or PET) or C0G / NP0"
- note added: "ICS-40730 Output Impedance: 430 Ohm differential"
- note added: "R analog sound: Thin Film / Metal Film (Recommended)"
- note added: "Rf"
- note added: "Rg"
- note removed: "1% Tolerance Resistors"
- note removed: "2. Dielectric Absorption (Ceramic Capacitor Distortions) This is where the "special" capacitor conversation actually matters. If you use cheap X7R or Z5U ceramic capacitors in the signal path, they change their capacitance as the voltage changes. This creates a non-linear distortion that can sound like graininess or crackling during loud bass notes. The Fix: For any capacitor actually touching th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"
- note removed: "Pins A0 and A1 are latched at start. The A0 pin is then used to alllow EEPROM write"
- moved on the sheet: C10, C2, C32, C7, C8, C9, MK1, MK2

Commit message: Update
Other:
- note added: "ICS-40730: Output Impedance: - OUTPUT+ is 180 Ohms - OUTPUT- is 250 Ohms - Differential is 430 Ohms Frequency Response: - From 20 Hz to 20 kHz Maximum Output Voltage: - Single-Ended, 123 dB SPL input is 0.40V rms This is Vpp≈1.13 V. Output DC Offset: - OUTPUT+ is 0.72V - OUTPUT- is 0.66V"
- note added: "R analog sound: Thin Film/Metal Film (Recommended)"
- note removed: "Frequency Response from 20 Hz to 20 kHz"
- note removed: "It is also possible to connect the VOCM input to a common-mode level (CML) output of an ADC. However, care must be taken to ensure that the output has sufficient drive capability. The input impedance of the VOCM pin is approximately 250 kΩ."
- note removed: "Maximum Output Voltage Single-Ended, 123 dB SPL input is 0.40V rms This is Vpp≈1.13 V."
- note removed: "Output DC Offset OUTPUT+ is 0.72V OUTPUT- is 0.66V"
- note removed: "Output Impedance OUTPUT+ is 180 Ohms OUTPUT- is 250 Ohms Differential is 430 Ohms"
- moved on the sheet: AMP1, C10, C2, C32, C39, C40, C41, C42, C43, C44, C45, C46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
