File: ADC_Driver_ADA4940-2ACPZ-R7.kicad_sch (KiCad schematic)
At the start: 29 parts

Commit message: Update
Changed lines of the file:
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@@
+		)
+	)
+	(text "length-matched"
+		(exclude_from_sim no)
+		(at 242.316 74.422 0)
+		(effects
+			(font
+				(size 1 1)
+			)
 		)
 	)
@@
 		(effects
 			(font
+				(size 1 1)
+			)
+		)
+	)
+	(text "length-matched"
+		(exclude_from_sim no)
+		(at 98.552 145.796 0)
+		(effects
+			(font
+				(size 1 1)
+			)
+		)
+	)
+	(text "length-matched"
+		(exclude_from_sim no)
+		(at 235.712 130.048 0)
+		(effects
+			(font

Commit message: Update
Other:
- note added: "R analog sound: Thin Film/Metal Film (Recommended) Rg variable"
- note removed: "R analog sound: Thin Film/Metal Film (Recommended)"
Changed lines of the file:
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@@
 		)
 	)
-	(text "R analog sound: \nThin Film/Metal Film (Recommended)"
+	(text "R analog sound: \nThin Film/Metal Film (Recommended)\nRg variable"
 		(exclude_from_sim no)
-		(at 98.552 55.88 0)
+		(at 103.632 55.118 0)
 		(effects
 			(font

Commit message: Update
Parts:
- removed C32: 10u, Capacitor_SMD:C_0805_2012Metric, symbol Device:C
- added C25: 10u, Capacitor_SMD:C_1812_4532Metric, symbol Device:C
- C10, C8, C9: footprint Capacitor_SMD:C_0805_2012Metric -> Capacitor_SMD:C_1812_4532Metric
- C39, C41, C43, C44: footprint Capacitor_SMD:C_0805_2012Metric -> Capacitor_SMD:C_0603_1608Metric
- C40, C42: value 100n -> 1n; footprint Capacitor_SMD:C_0805_2012Metric -> Capacitor_SMD:C_0603_1608Metric
- R18, R19, R26, R27: value 1K_RN73H2ATTD1001B25 -> 1k
- R28, R29: value 22R -> 33R
- R30, R31: value 22R_Metal_Film -> 33R
Connections:
- net MIC_R_C_OUT-: now also C25.2
- net MIC_R_OUT-: now also C25.1
- net +OUT1 renamed OUT1+
- net +OUT2 renamed OUT2+
- net -OUT1 renamed OUT1-
- net -OUT2 renamed OUT2-
Other:
- note added: "Film Capacitors (PPS or PET) or C0G / NP0 Bipolar Aluminum Electrolytic Good Polyester Film (MKT) Best"
- note removed: "Film Capacitors (PPS or PET) or C0G / NP0"
