File: ADC_Driver_ADA4940-2ACPZ-R7.kicad_sch (KiCad schematic)
At the start: 29 parts

Commit message: Update
Parts:
- C10, C25, C8, C9: value 10u -> 10u_16MU106MC44532
Other:
- note added: "ADI ADA4940-1ARZ"
- note added: "ALT: ICS-40720 (DK), ICS-40740 (Mouser)"
- moved on the sheet: C10, C25, C7, MK2
