File: Notes.kicad_sch (KiCad schematic)
At the start: 0 parts

Commit message: Update
Changed lines of the file:
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@@
 	(generator_version "8.0")
 	(paper "USLetter")
-	(text_box "Notes:\n- Physical power inputs: 3V3, 5V\n- Power Consumption\n  CS5381K-KSZ\n  - IA = 50mA, ID = 50mA, ID = 30mA (MAX), ITOTAL = 130mA\n  ADC_Driver_ADA4940-2ACPZ-R7\n  - I = 2.5mA\n  Microphones\n  - I = 1mA\n  -----------\n  Device Total 150mA\n\n- All power inputs include polarity protection\n- Will be using 12.288 MHz to cover all possible conversion rates of CS5381\n- VA Analog MIN is 4.25V to 5.25V (Should be 5V)\n- VD Digital MIN is 3.1V to 5.25V\n- VL Logic MIN is 237V to 5.25V\n- VD pin powers the chip's digital core logic - the internal digital processing circuitry that handles things like:\n  (Delta-sigma modulator output, Digital filters (decimation, etc.), Sample rate control logic, Configuration control logic (I²C/SPI core))\n- VL (Logic 1 = VL) controls MCLK, SCLK, LRCK\n- Power from USB: pins D+/D- left optionally floating or shorted\n\nFullscale Input Level = (Ain+)-(Ain-) = 5.64 Vpp\nAin+ is between 3.91 and 1.09 V (Each leg swinging 2.82V)\nAin- is between 3.91 and 1.09 V\nBoth oscillate around 2.5V (Common mode level)\nThe DC bias (Common mode level) is sett using VQ or VCOM (one pin)\nVQ or VCOM nominal voltage is 2.5V\nFilt+ Nominal Voltage 5V (Positive voltage reference output)\n\n- To reach 2.82 Vpp differential at the ADC:\nRequired gain\nG≈2.82/2.26≈1.25 per leg (use two identical amps).\nDifferential Vpp scales by the same per-leg gain if both paths are equal.\nIf your target were 2.82 Vpp per input (single-ended):\nG≈2.82/1.13≈2.5 per leg.\n\nImpedance Matching between Microphone and ADA4940\n- Output Impedance to ICS-40730 is 430 Ohms\n- Input Differential Impedance to ADA4940-2 is Rin = 2 x 200 Ohms = 400 Ohms"
+	(text_box "Notes:\n- Physical power inputs: 3V3, 5V\n- Power Consumption\n  CS5381K-KSZ\n  - IA = 50mA, ID = 50mA, ID = 30mA (MAX), ITOTAL = 130mA\n  ADC_Driver_ADA4940-2ACPZ-R7\n  - I = 2.5mA\n  Microphones\n  - I = 1mA\n  -----------\n  Device Total 150mA\n\n- All power inputs include polarity protection\n- Will be using 12.288 MHz to cover all possible conversion rates of CS5381\n- VA Analog MIN is 4.25V to 5.25V (Should be 5V)\n- VD Digital MIN is 3.1V to 5.25V\n- VL Logic MIN is 237V to 5.25V\n- VD pin powers the chip's digital core logic - the internal digital processing circuitry that handles things like:\n  (Delta-sigma modulator output, Digital filters (decimation, etc.), Sample rate control logic, Configuration control logic (I²C/SPI core))\n- VL (Logic 1 = VL) controls MCLK, SCLK, LRCK\n- Power from USB: pins D+/D- left optionally floating or shorted\n\nFullscale Input Level = (Ain+)-(Ain-) = 5.64 Vpp\nAin+ is between 3.91 and 1.09 V (Each leg swinging 2.82V)\nAin- is between 3.91 and 1.09 V\nBoth oscillate around 2.5V (Common mode level)\nThe DC bias (Common mode level) is sett using VQ or VCOM (one pin)\nVQ or VCOM nominal voltage is 2.5V\nFilt+ Nominal Voltage 5V (Positive voltage reference output)\n\n- To reach 2.82 Vpp differential at the ADC:\nRequired gain\nG≈2.82/2.26≈1.25 per leg (use two identical amps).\nDifferential Vpp scales by the same per-leg gain if both paths are equal.\nIf your target were 2.82 Vpp per input (single-ended):\nG≈2.82/1.13≈2.5 per leg.\n\nImpedance Matching between Microphone and ADA4940\n- Output Impedance to ICS-40730 is 430 Ohms\n- Input Differential Impedance to ADA4940-2 is Rin = 2 x 200 Ohms = 400 Ohms\n- The input impedance (dif) of ADA4940 should be 10x of souurce impedance\n  - 10x 430 = 4k3 Ohms therefore make each Rg=2k"
 		(exclude_from_sim no)
 		(at 26.035 26.035 0)

Commit message: Update
Changed lines of the file:
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@@
 	(generator_version "8.0")
 	(paper "USLetter")
+	(text_box "NOTES:\nCS5381K-KSZ Turn OFF or LOW Power mode\n- CS5381K-KSZ enters LOW power mode when RST pin LOW\n- CS5381K-KSZ cannot be connected to GLOBAL RST because it is used to enter LOW power mode meaning it does not function as device RST\n- PU R is placed in the CS5381K-KSZ RST\n\nOVFL pin is open drain\nWhen no overflow detected\nthe pin will be HIGH.\nWhen overflow detected\nthe pin will be LOW\n\nHPF High Pass Filter inside CS5381K-KSZ\n- To remove DC offset\n- To be run initially then disabled\n- Value is frozen and used thereafter "
+		(exclude_from_sim no)
+		(at 25.908 122.682 0)
+		(size 100.33 69.85)
+		(stroke
+			(width 0)
+			(type dash)
+		)
+		(fill
+			(type none)
+		)
+		(effects
+			(font
+				(size 1 1)
+			)
+			(justify left top)
+		)
+	)
 	(text_box "Notes:\n- Physical power inputs: 3V3, 5V\n- Power Consumption\n  CS5381K-KSZ\n  - IA = 50mA, ID = 50mA, ID = 30mA (MAX), ITOTAL = 130mA\n  ADC_Driver_ADA4940-2ACPZ-R7\n  - I = 2.5mA\n  Microphones\n  - I = 1mA\n  -----------\n  Device Total 150mA\n\n- All power inputs include polarity protection\n- Will be using 12.288 MHz to cover all possible conversion rates of CS5381\n- VA Analog MIN is 4.25V to 5.25V (Should be 5V)\n- VD Digital MIN is 3.1V to 5.25V\n- VL Logic MIN is 237V to 5.25V\n- VD pin powers the chip's digital core logic - the internal digital processing circuitry that handles things like:\n  (Delta-sigma modulator output, Digital filters (decimation, etc.), Sample rate control logic, Configuration control logic (I²C/SPI core))\n- VL (Logic 1 = VL) controls MCLK, SCLK, LRCK\n- Power from USB: pins D+/D- left optionally floating or shorted\n\nFullscale Input Level = (Ain+)-(Ain-) = 5.64 Vpp\nAin+ is between 3.91 and 1.09 V (Each leg swinging 2.82V)\nAin- is between 3.91 and 1.09 V\nBoth oscillate around 2.5V (Common mode level)\nThe DC bias (Common mode level) is sett using VQ or VCOM (one pin)\nVQ or VCOM nominal voltage is 2.5V\nFilt+ Nominal Voltage 5V (Positive voltage reference output)\n\n- To reach 2.82 Vpp differential at the ADC:\nRequired gain\nG≈2.82/2.26≈1.25 per leg (use two identical amps).\nDifferential Vpp scales by the same per-leg gain if both paths are equal.\nIf your target were 2.82 Vpp per input (single-ended):\nG≈2.82/1.13≈2.5 per leg.\n\nImpedance Matching between Microphone and ADA4940\n- Output Impedance to ICS-40730 is 430 Ohms\n- Input Differential Impedance to ADA4940-2 is Rin = 2 x 200 Ohms = 400 Ohms\n- The input impedance (dif) of ADA4940 should be 10x of souurce impedance\n  - 10x 430 = 4k3 Ohms therefore make each Rg=2k"
 		(exclude_from_sim no)
@@
 		(effects
 			(font
-				(size 1.27 1.27)
+				(size 1 1)
 			)
 			(justify left top)
@@
 		(effects
 			(font
-				(size 1.27 1.27)
+				(size 1 1)
 			)
 			(justify left top)
@@
 	(text "Fullscale Input Level = (Ain+)-(Ain-) = 5.64 Vpp\nAin+ is between 3.91 and 1.09 V (Each leg swinging 2.82V)\nAin- is between 3.91 and 1.09 V\nBoth oscillate around 2.5V (Common mode level)\nThe DC bias (Common mode level) is sett using VQ or VCOM (one pin)\nVQ or VCOM nominal voltage is 2.5V\nFilt+ Nominal Voltage 5V (Positive voltage reference output)"
 		(exclude_from_sim no)
-		(at 33.528 132.08 0)
+		(at 160.274 133.096 0)
 		(effects
 			(font
